File: Parent_Turtle_ver.servo_main_ver.4/Parent_Turtle_Servo.kicad_pcb (KiCad board)
At the start: 2 copper layers, 70 x 60 mm, 61 parts, among them P1 CONN_02X15, P10 WRITING, P11 A/D, P12 5V_in, P13 CONN_02X04, P14 I/O, P15 CONN_02X04, P16 PWM, P17 SERIAL0, P2 CONN_02X15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

Commit message: Add Parent Turtle ver.4, ver.5
Parts:
- C6, C7: moved to B.Cu
- moved C6 45.5 mm to (165.8, 105.2)
- moved C7 41.3 mm to (168.9, 114.6)
- moved U3 8.90 mm to (166.6, 109.4)
Routing:
- net +5V: track 108.4 -> 171.7 mm
- net +12V: track 11.3 -> 19.7 mm
Changed lines of the file:
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@@
   (general
     (links 154)
-    (no_connects 13)
-    (area 101.014999 69.584999 171.165001 129.735001)
+    (no_connects 4)
+    (area 97.889999 16.04 279.593333 133.358333)
     (thickness 1.6)
     (drawings 13)
-    (tracks 432)
+    (tracks 456)
     (zones 0)
     (modules 61)
@@
   )
   (setup
-    (last_trace_width 0.3)
+    (last_trace_width 0.25)
     (user_trace_width 0.3)
     (user_trace_width 0.5)
@@
       (drillshape 0)
       (scaleselection 1)
-      (outputdirectory ../加工データ/Servo_main/))
+      (outputdirectory E:/Servo_main/))
   )
   (net 0 "")
@@
     )
   )
-  (module Capacitors_SMD:C_0603 (layer F.Cu)
-    (at 136.09 139.735001)
+  (module Capacitors_SMD:C_0603 (layer B.Cu)
+    (at 165.77 105.24)
     (descr "Capacitor SMD 0603, reflow soldering, AVX (see smccp.pdf)")
     (tags "capacitor 0603")
     (attr smd)
-    (fp_text reference C6 (at 0 -1.9) (layer F.SilkS)
-      (effects (font (size 1 1) (thickness 0.15)))
-    )
-    (fp_text value 0.1u (at 0 1.9) (layer F.Fab)
-      (effects (font (size 1 1) (thickness 0.15)))
-    )
-    (fp_line (start -0.8 0.4) (end -0.8 -0.4) (layer F.Fab) (width 0.15))
-    (fp_line (start 0.8 0.4) (end -0.8 0.4) (layer F.Fab) (width 0.15))
-    (fp_line (start 0.8 -0.4) (end 0.8 0.4) (layer F.Fab) (width 0.15))
-    (fp_line (start -0.8 -0.4) (end 0.8 -0.4) (layer F.Fab) (width 0.15))
-    (fp_line (start -1.45 -0.75) (end 1.45 -0.75) (layer F.CrtYd) (width 0.05))
-    (fp_line (start -1.45 0.75) (end 1.45 0.75) (layer F.CrtYd) (width 0.05))
-    (fp_line (start -1.45 -0.75) (end -1.45 0.75) (layer F.CrtYd) (width 0.05))
-    (fp_line (start 1.45 -0.75) (end 1.45 0.75) (layer F.CrtYd) (width 0.05))
-    (fp_line (start -0.35 -0.6) (end 0.35 -0.6) (layer F.SilkS) (width 0.15))
-    (fp_line (start 0.35 0.6) (end -0.35 0.6) (layer F.SilkS) (width 0.15))
-    (pad 1 smd rect (at -0.95 0) (size 1 1.2) (layers F.Cu F.Paste F.Mask)
+    (fp_text reference C6 (at 0 1.9) (layer B.SilkS)
+      (effects (font (size 1 1) (thickness 0.15)) (justify mirror))
+    )
+    (fp_text value 0.1u (at 0 -1.9) (layer B.Fab)
+      (effects (font (size 1 1) (thickness 0.15)) (justify mirror))
+    )
+    (fp_line (start -0.8 -0.4) (end -0.8 0.4) (layer B.Fab) (width 0.15))
+    (fp_line (start 0.8 -0.4) (end -0.8 -0.4) (layer B.Fab) (width 0.15))
+    (fp_line (start 0.8 0.4) (end 0.8 -0.4) (layer B.Fab) (width 0.15))
+    (fp_line (start -0.8 0.4) (end 0.8 0.4) (layer B.Fab) (width 0.15))
+    (fp_line (start -1.45 0.75) (end 1.45 0.75) (layer B.CrtYd) (width 0.05))
+    (fp_line (start -1.45 -0.75) (end 1.45 -0.75) (layer B.CrtYd) (width 0.05))
+    (fp_line (start -1.45 0.75) (end -1.45 -0.75) (layer B.CrtYd) (width 0.05))
+    (fp_line (start 1.45 0.75) (end 1.45 -0.75) (layer B.CrtYd) (width 0.05))
+    (fp_line (start -0.35 0.6) (end 0.35 0.6) (layer B.SilkS) (width 0.15))
+    (fp_line (start 0.35 -0.6) (end -0.35 -0.6) (layer B.SilkS) (width 0.15))
+    (pad 1 smd rect (at -0.95 0) (size 1 1.2) (layers B.Cu B.Paste B.Mask)
       (net 69 +12V))
-    (pad 2 smd rect (at 0.93 0) (size 1 1.2) (layers F.Cu F.Paste F.Mask)
+    (pad 2 smd rect (at 0.93 0) (size 1 1.2) (layers B.Cu B.Paste B.Mask)
       (net 2 GND))
     (model Capacitors_SMD.3dshapes/C_0603.wrl
@@
     )
   )
-  (module Capacitors_SMD:C_0603 (layer F.Cu)
-    (at 136.09 139.735001)
+  (module Capacitors_SMD:C_0603 (layer B.Cu)
+    (at 168.95 114.64)
     (descr "Capacitor SMD 0603, reflow soldering, AVX (see smccp.pdf)")
     (tags "capacitor 0603")
     (attr smd)
-    (fp_text reference C7 (at 0 -1.9) (layer F.SilkS)
-      (effects (font (size 1 1) (thickness 0.15)))
-    )
-    (fp_text value 0.1u (at 0 1.9) (layer F.Fab)
-      (effects (font (size 1 1) (thickness 0.15)))
-    )
-    (fp_line (start -0.8 0.4) (end -0.8 -0.4) (layer F.Fab) (width 0.15))
-    (fp_line (start 0.8 0.4) (end -0.8 0.4) (layer F.Fab) (width 0.15))
-    (fp_line (start 0.8 -0.4) (end 0.8 0.4) (layer F.Fab) (width 0.15))
-    (fp_line (start -0.8 -0.4) (end 0.8 -0.4) (layer F.Fab) (width 0.15))
-    (fp_line (start -1.45 -0.75) (end 1.45 -0.75) (layer F.CrtYd) (width 0.05))
-    (fp_line (start -1.45 0.75) (end 1.45 0.75) (layer F.CrtYd) (width 0.05))
-    (fp_line (start -1.45 -0.75) (end -1.45 0.75) (layer F.CrtYd) (width 0.05))
-    (fp_line (start 1.45 -0.75) (end 1.45 0.75) (layer F.CrtYd) (width 0.05))
-    (fp_line (start -0.35 -0.6) (end 0.35 -0.6) (layer F.SilkS) (width 0.15))
-    (fp_line (start 0.35 0.6) (end -0.35 0.6) (layer F.SilkS) (width 0.15))
-    (pad 1 smd rect (at -0.95 0) (size 1 1.2) (layers F.Cu F.Paste F.Mask)
+    (fp_text reference C7 (at 0 1.9) (layer B.SilkS)
+      (effects (font (size 1 1) (thickness 0.15)) (justify mirror))
+    )
+    (fp_text value 0.1u (at 0 -1.9) (layer B.Fab)
+      (effects (font (size 1 1) (thickness 0.15)) (justify mirror))
+    )
+    (fp_line (start -0.8 -0.4) (end -0.8 0.4) (layer B.Fab) (width 0.15))
+    (fp_line (start 0.8 -0.4) (end -0.8 -0.4) (layer B.Fab) (width 0.15))
+    (fp_line (start 0.8 0.4) (end 0.8 -0.4) (layer B.Fab) (width 0.15))
+    (fp_line (start -0.8 0.4) (end 0.8 0.4) (layer B.Fab) (width 0.15))
+    (fp_line (start -1.45 0.75) (end 1.45 0.75) (layer B.CrtYd) (width 0.05))
+    (fp_line (start -1.45 -0.75) (end 1.45 -0.75) (layer B.CrtYd) (width 0.05))
+    (fp_line (start -1.45 0.75) (end -1.45 -0.75) (layer B.CrtYd) (width 0.05))
+    (fp_line (start 1.45 0.75) (end 1.45 -0.75) (layer B.CrtYd) (width 0.05))
+    (fp_line (start -0.35 0.6) (end 0.35 0.6) (layer B.SilkS) (width 0.15))
+    (fp_line (start 0.35 -0.6) (end -0.35 -0.6) (layer B.SilkS) (width 0.15))
+    (pad 1 smd rect (at -0.95 0) (size 1 1.2) (layers B.Cu B.Paste B.Mask)
       (net 1 +5V))
-    (pad 2 smd rect (at 0.93 0) (size 1 1.2) (layers F.Cu F.Paste F.Mask)
+    (pad 2 smd rect (at 0.93 0) (size 1 1.2) (layers B.Cu B.Paste B.Mask)
       (net 2 GND))
     (model Capacitors_SMD.3dshapes/C_0603.wrl
@@
   )
   (module TO_SOT_Packages_SMD:SOT89-3_Housing (layer B.Cu)
-    (at 175.5 108.5)
+    (at 166.64 109.36)
     (descr "SOT89-3, Housing,")
     (tags "SOT89-3, Housing,")
@@
   (via (at 168.09 126.66) (size 6) (drill 3) (layers F.Cu B.Cu) (net 0))
   (via (at 104.09 126.66) (size 6) (drill 3) (layers F.Cu B.Cu) (net 0))
+  (segment (start 168 114.64) (end 168 119.5) (width 0.5) (layer B.Cu) (net 1))
+  (segment (start 165.04 123.86) (end 163.19 125.71) (width 0.5) (layer B.Cu) (net 1))
+  (segment (start 165.04 122.46) (end 165.04 123.86) (width 0.5) (layer B.Cu) (net 1))
+  (segment (start 168 119.5) (end 165.04 122.46) (width 0.5) (layer B.Cu) (net 1))
+  (segment (start 163.19 125.71) (end 162.37 125.71) (width 0.5) (layer B.Cu) (net 1))
+  (segment (start 168.14114 107.50834) (end 168.14114 108.26114) (width 0.5) (layer B.Cu) (net 1))
+  (segment (start 168 113.14) (end 168 114.64) (width 0.5) (layer B.Cu) (net 1))
+  (segment (start 168.69 112.45) (end 168 113.14) (width 0.5) (layer B.Cu) (net 1))
+  (segment (start 168.69 108.81) (end 168.69 112.45) (width 0.5) (layer B.Cu) (net 1))
+  (segment (start 168.14114 108.26114) (end 168.69 108.81) (width 0.5) (layer B.Cu) (net 1))
+  (segment (start 168.14114 107.50834) (end 168.14114 103.95114) (width 0.5) (layer B.Cu) (net 1))
+  (segment (start 154.49 75.5) (end 151.75 75.5) (width 0.5) (layer B.Cu) (net 1))
+  (segment (start 158.2 79.21) (end 154.49 75.5) (width 0.5) (layer B.Cu) (net 1))
+  (segment (start 158.2 85.72) (end 158.2 79.21) (width 0.5) (layer B.Cu) (net 1))
+  (segment (start 160.18 87.7) (end 158.2 85.72) (width 0.5) (layer B.Cu) (net 1))
+  (segment (start 162.43 87.7) (end 160.18 87.7) (width 0.5) (layer B.Cu) (net 1))
+  (segment (start 165.75 91.02) (end 162.43 87.7) (width 0.5) (layer B.Cu) (net 1))
+  (segment (start 165.75 101.56) (end 165.75 91.02) (width 0.5) (layer B.Cu) (net 1))
+  (segment (start 168.14114 103.95114) (end 165.75 101.56) (width 0.5) (layer B.Cu) (net 1))
   (segment (start 162.37 125.71) (end 162.71 125.71) (width 0.5) (layer B.Cu) (net 1))
   (segment (start 159.83 125.71) (end 162.37 125.71) (width 0.5) (layer B.Cu) (net 1))
@@
   (segment (start 152.97 90.22) (end 152.97 95.06) (width 0.3) (layer B.Cu) (net 68))
   (segment (start 154.61 89.79) (end 154.59 89.77) (width 0.3) (layer B.Cu) (net 68))
+  (segment (start 164.82 105.24) (end 164.82 107.18948) (width 0.5) (layer B.Cu) (net 69))
+  (segment (start 164.82 107.18948) (end 165.13886 107.50834) (width 0.5) (layer B.Cu) (net 69))
+  (segment (start 161.58 101.81) (end 163.6 101.81) (width 0.5) (layer B.Cu) (net 69))
+  (segment (start 164.82 103.03) (end 164.82 105.24) (width 0.5) (layer B.Cu) (net 69))
+  (segment (start 163.6 101.81) (end 164.82 103.03) (width 0.5) (layer B.Cu) (net 69))
   (segment (start 150.6 100.99) (end 153.71 100.99) (width 0.5) (layer B.Cu) (net 69))
   (segment (start 153.71 100.99) (end 154.46 101.74) (width 0.5) (layer B.Cu) (net 69))
