File: Parent_Turtle_ver.servo_main_ver.4/Parent_Turtle_Servo.sch (KiCad schematic (older format))
At the start: 61 parts, among them P1 CONN_02X15, P10 WRITING, P11 A/D, P12 5V_in, P13 CONN_02X04, P14 I/O, P15 CONN_02X04, P16 PWM, P17 SERIAL0, P2 CONN_02X15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

Commit message: そういえば，RC19の基板整理していなかった(リポジトリ的にも)
Parts:
- C1, C2, C3, C4, C5, C6, C7: symbol C -> Parent_Turtle_Servo-rescue:C
- D1, D10, D11, D2, D3, D4, D5, D6, D7, D8, D9: symbol LED -> Parent_Turtle_Servo-rescue:LED
- D12: symbol DIODE -> Parent_Turtle_Servo-rescue:DIODE
- P1, P2: symbol CONN_02X15 -> Parent_Turtle_Servo-rescue:CONN_02X15
- P10: symbol CONN_01X06 -> Parent_Turtle_Servo-rescue:CONN_01X06
- P11, P14, P17, P3, P4, P7, P8: symbol CONN_01X04 -> Parent_Turtle_Servo-rescue:CONN_01X04
- P12, P16, P9: symbol CONN_01X02 -> Parent_Turtle_Servo-rescue:CONN_01X02
- P13, P15: symbol CONN_02X04 -> Parent_Turtle_Servo-rescue:CONN_02X04
- P5: symbol CONN_01X14 -> Parent_Turtle_Servo-rescue:CONN_01X14
- P6: symbol USB_OTG -> Parent_Turtle_Servo-rescue:USB_OTG
- Q1: symbol NPN -> Parent_Turtle_Servo-rescue:NPN
- R1, R10, R11, R12, R13, R14, R15, R16, R17, R18, R2, R3, R4, R5, R6, R7, R8, R9: symbol R -> Device:R
- SP1: symbol SPEAKER -> Parent_Turtle_Servo-rescue:SPEAKER
- SW1, SW2: symbol SW_PUSH -> Parent_Turtle_Servo-rescue:SW_PUSH
- U1: symbol MAX3051 -> Parent_Turtle_Servo-rescue:MAX3051
- U2: symbol MCP2221 -> Parent_Turtle_Servo-rescue:MCP2221
- U3: symbol 78L05 -> Parent_Turtle_Servo-rescue:78L05
