File: Parent_Turtle_ver.servo_main_ver.5/Parent_Turtle_RC19main.sch (KiCad schematic (older format))
At the start: 65 parts, among them P1 CONN_02X15, P10 WRITING, P11 A/D, P12 5V_in, P13 CONN_02X04, P14 I/O, P15 CONN_02X04, P16 PWM, P17 SERIAL0, P2 CONN_02X15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

Commit message: クランリンケージ用main基板完成版
Parts:
- removed D7, D8: LED, LEDs:LED-3MM, symbol LED
- removed P16: PWM, Pin_Headers:Pin_Header_Straight_1x02, symbol CONN_01X02
- removed P5: PWM, Pin_Headers:Pin_Header_Straight_1x14, symbol CONN_01X14
- removed P? (x3): ENC, symbol CONN_01X04
- removed R12, R13: 330, Resistors_SMD:R_0603, symbol R
- removed U3: 78L05, TO_SOT_Packages_SMD:SOT89-3_Housing, symbol 78L05
- added C10, C11, C8, C9: 0.1u, Capacitors_SMD:C_0603, symbol C
- added D13, D14: DIODE, Mizz_lib:SOD-123, symbol DIODE
- added L1: 10uH, Inductors:Inductor_Wurth_MAPI-2512, symbol INDUCTOR
- added P19, P20, P21: ENC, RP_KiCAD_Connector:XA_4T, symbol CONN_01X04
- added P5: PWM, Pin_Headers:Pin_Header_Straight_1x08, symbol CONN_01X08
- added R19, R20, R21, R22, R27, R28, R29, R30: 100, Resistors_SMD:R_0603, symbol R
- added R23, R24, R25, R26, R31, R32, R33, R34: 1k, Resistors_SMD:R_0603, symbol R
- added R35: 50k, Resistors_SMD:R_0603, symbol R
- added R36: 10k, Resistors_SMD:R_0603, symbol R
- added U3: AOZ1280, Mizz_lib:TSOT-6-MK06A, symbol AOZ1280
- C7: value 0.1u -> 1u
- P11: value A/D -> ADC
- P13: value CONN_02X04 -> ADC/Vdd/GND
- P15: value CONN_02X04 -> I/O /Vdd/GND
- P18: renamed from P?; footprint (none) -> RP_KiCAD_Connector:XA_4T
Connections:
- net +12V: now also C7.1, U3.4 (EN), U3.5 (VIN); no longer C6.1
- net +3.3V: now also R23.2, R24.2, R25.2, R26.2, R31.2, R32.2, R33.2, R34.2
- net +5V: now also P18.2 (P2), C10.1, C11.1, C8.1, C9.1, D14.2 (K), P19.2 (P2), P20.2 (P2), P21.2 (P2); no longer C7.1
- net A0: now also R27.2
- net A1: now also R28.2
- net A6: now also R19.2
- net A7: now also R20.2
- net A8: now also R4.1
- net B15: now also P14.3 (P3)
- net B7: now also R7.2, SW2.2
- net B8: now also R2.2, SW1.2
- net C6: now also R11.1; no longer R4.1
- net D12: now also R21.2
- net D13: now also R22.2; no longer P14.2 (P2)
- net D15: no longer P14.1 (P1), R11.1
- net D8: now also P14.1 (P1)
- net D9: now also P14.2 (P2); no longer P14.3 (P3)
- net E10: no longer R7.2, SW2.2
- net E12: no longer R2.2, SW1.2
- net E5: now also R29.2
- net E6: now also R30.2
- net GND: now also P18.1 (P1), C10.2, C11.2, C8.2, C9.2, D13.1 (A), P19.1 (P1), P20.1 (P1), P21.1 (P1), R36.1, U3.2 (GND); no longer C6.2
- net at P18.3 (P3): now also R19.1, R23.1
- net at P18.4 (P4): now also R20.1, R25.1
- new net: P20.3 (P3), R27.1, R31.1
- new net: P20.4 (P4), R28.1, R33.1
- new net: P19.3 (P3), R21.1, R24.1
- new net: P19.4 (P4), R22.1, R26.1
- new net: P21.3 (P3), R29.1, R32.1
- new net: P21.4 (P4), R30.1, R34.1
- new net: C6.2, U3.1 (BST)
- new net: C6.1, D13.2 (K), L1.1, U3.6 (LX)
- new net: D14.1 (A), L1.2, R35.2
- new net FB: R35.1, R36.2, U3.3 (FB)
Other:
- note added: "http://akizukidenshi.com/catalog/g/gP-06984/"
- moved on the sheet: C2, C3, C5, D10, D11, P11, P13, P14, P15, P17, P18, P6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

Commit message: ver.5は本当にこれが完成版.
Parts:
- P18: value ENC -> ENC2
- P19: value ENC -> ENC3
- P20: value ENC -> ENC1
- P21: value ENC -> ENC0
Changed lines of the file:
@@
 P 2150 1950
 F 0 "P18" H 2150 2200 50  0000 C CNN
-F 1 "ENC" V 2250 1950 50  0000 C CNN
+F 1 "ENC2" V 2250 1950 50  0000 C CNN
 F 2 "RP_KiCAD_Connector:XA_4T" H 2150 1950 50  0001 C CNN
 F 3 "" H 2150 1950 50  0000 C CNN
@@
 P 3350 1950
 F 0 "P20" H 3350 2200 50  0000 C CNN
-F 1 "ENC" V 3450 1950 50  0000 C CNN
+F 1 "ENC1" V 3450 1950 50  0000 C CNN
 F 2 "RP_KiCAD_Connector:XA_4T" H 3350 1950 50  0001 C CNN
 F 3 "" H 3350 1950 50  0000 C CNN
@@
 P 2150 2925
 F 0 "P19" H 2150 3175 50  0000 C CNN
-F 1 "ENC" V 2250 2925 50  0000 C CNN
+F 1 "ENC3" V 2250 2925 50  0000 C CNN
 F 2 "RP_KiCAD_Connector:XA_4T" H 2150 2925 50  0001 C CNN
 F 3 "" H 2150 2925 50  0000 C CNN
@@
 P 3350 2925
 F 0 "P21" H 3350 3175 50  0000 C CNN
-F 1 "ENC" V 3450 2925 50  0000 C CNN
+F 1 "ENC0" V 3450 2925 50  0000 C CNN
 F 2 "RP_KiCAD_Connector:XA_4T" H 3350 2925 50  0001 C CNN
 F 3 "" H 3350 2925 50  0000 C CNN
