File: Parent_Turtle_ver.servo_main_ver.5/Parent_Turtle_RC19main.sch (KiCad schematic (older format))
At the start: 89 parts, among them P1 CONN_02X15, P10 WRITING, P11 ADC, P12 5V_in, P13 ADC/Vdd/GND, P14 I/O, P15 I/O /Vdd/GND, P17 SERIAL0, P18 ENC2, P19 ENC3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

Commit message: インダクタのフットプリントの修正.
Parts:
- L1: footprint Inductors_NEOSID:Neosid_Inductor_Ms50 -> Inductors:Inductor_Taiyo-Yuden_NR-50xx_HandSoldering
Changed lines of the file:
@@
 F 0 "L1" V 5200 950 40  0000 C CNN
 F 1 "10uH" V 5350 950 40  0000 C CNN
-F 2 "Inductors_NEOSID:Neosid_Inductor_Ms50" H 5250 950 60  0001 C CNN
+F 2 "Inductors:Inductor_Taiyo-Yuden_NR-50xx_HandSoldering" H 5250 950 60  0001 C CNN
 F 3 "" H 5250 950 60  0000 C CNN
 	1    5250 950
