File: stm32f4-cosmos/stm32f4_cosmos/stm32f4_cosmos.kicad_pcb (KiCad board)
At the start: 2 copper layers, 100 x 94 mm, 191 parts, among them IC1 PIC24FJ64GB004, P1 PICKit3, P10 5V, P11 CAN0, P12 CAN1, P13 CAN0, P14 CAN1, P15 SERIAL, P16 SERIAL, P17 12V, P18 SWD, P2 SBDBT, P23 A/D, P24 PWM, P25 A/D_batt, P26 PWM_batt, P27 EMERGENCY_CHECK, P28 I/O_3.3V, P29 I/O_5V, P3 ENC, P30 I/O_3.3V_batt, P31 I/O_5V_batt, P4 ENC, P5 SERIALx, P6 ENC, P7 ENC, P8 SERIAL, P9 SERIAL, Q1 P_FET, Q2 P_FET, Q3 P_FET, Q4 NPN, Q5 NPN, SW1 POWER_ON, SW2 SW1, SW3 SW0, SW4 SW2, SW5 SW3, U1 STM32F407VG, U10 LOGO, U11 LOGO, U12 25LC010A, U2 AZ1086H, U3 MCP2221A, U4 AP3211, U5 MAX3051, U6 MAX3051, U7 AQM1602_BL, U8 OSTBABS4C2B, U9 LOGO, X1 8MHz

Commit message: 良い感じ.
Parts:
- D18: value CAN_BUS_12V -> 12V
- moved D10 99.8 mm to (113.5, 160.2), turned to 180 degrees
- moved R30 95.5 mm to (110.8, 160.2), turned to 180 degrees
- moved D9 79.6 mm to (93.0, 152.0), turned to 180 degrees
- moved R29 75.8 mm to (90.5, 152.0), turned to 180 degrees
- moved R26 51.2 mm to (79.5, 111.8)
- moved R27 51.2 mm to (79.5, 114.8)
- moved R28 51.2 mm to (79.5, 108.8)
- moved D6 50.9 mm to (77.0, 111.8)
- moved D7 50.9 mm to (77.0, 114.8)
- moved D8 50.9 mm to (77.0, 108.8)
- moved R31 50.6 mm to (79.5, 105.8)
- moved D11 50.4 mm to (77.0, 105.8)
- moved R44 44.6 mm to (59.0, 128.5)
- moved D18 44.4 mm to (56.5, 128.5)
- moved R22 5.88 mm to (90.6, 127.9)
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Connections:
- D25 pad 1: /PA11 -> /PD0
- D3 pad 1: Net-(D3-Pad1) -> +3.3V
- D3 pad 2: GND -> Net-(D3-Pad2)
- D4 pad 1: Net-(D4-Pad1) -> +3.3V
- D4 pad 2: GND -> Net-(D4-Pad2)
- D5 pad 1: Net-(D5-Pad1) -> +3.3V
- D5 pad 2: GND -> Net-(D5-Pad2)
- R22 pad 1: Net-(D3-Pad1) -> Net-(D3-Pad2)
- R23 pad 1: Net-(D4-Pad1) -> Net-(D4-Pad2)
- R24 pad 1: Net-(D5-Pad1) -> Net-(D5-Pad2)
- R54 pad 2: /PA12 -> /PD1
- SW3 pad 2: /PA12 -> /PD1
- U1 pad 70: /PA11 -> /CAN1_RX
- U1 pad 71: /PA12 -> /CAN1_TX
- U1 pad 81: /CAN1_TX -> /PD0
- U1 pad 82: /CAN1_RX -> /PD1
- U12 pad 1: /PE7 -> /PE8
- U12 pad 3: /PE8 -> /PE7
Routing:
- net /I2C1_SCL: track 8.50 -> 100.9 mm, vias 1 -> 5
- net /I2C1_SDA: track 9.07 -> 99.2 mm, vias 1 -> 5
- net /NRST: track 39.8 -> 122.0 mm, vias 3 -> 8
- net +5V: track 285.1 -> 353.5 mm, vias 9 -> 12
- net /CAN1_RX: track 0.00 -> 54.8 mm, vias 0 -> 1
- net /USART2_RX: track 16.4 -> 71.0 mm, vias 0 -> 4
- net /CAN1_TX: track 0.00 -> 54.5 mm, vias 0 -> 1
- net /USART2_TX: track 14.8 -> 69.1 mm, vias 0 -> 4
- net +3.3V: track 416.2 -> 469.6 mm, vias 21 -> 29
- net /CAN2_RX: track 0.00 -> 48.8 mm, vias 0 -> 3
- net /CAN2_TX: track 0.00 -> 45.0 mm, vias 0 -> 1
- net /PD7: track 17.9 -> 59.0 mm, vias 0 -> 4
- net +12V: track 62.2 -> 101.0 mm, vias 0 -> 1
- net /PD10: track 0.00 -> 32.2 mm, vias 0 -> 2
- net /PD11: track 0.00 -> 29.8 mm, vias 0 -> 2
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
Commit message: あと四本.
Parts:
- added U13: LOGO, Mizz_lib:Enc_19.3x7.0_silk, F.Cu at (63.8, 58.5)
- R46, R47, R48: moved to F.Cu
- U11: footprint Mizz_lib:PPTP_CANT_silk_20x20 -> Mizz_lib:PPTP_uva_silk_20x18
- moved D10 58.5 mm to (77.0, 114.5), turned to 0 degrees
- moved R30 55.4 mm to (79.5, 114.5), turned to 0 degrees
- moved D9 38.0 mm to (77.0, 117.5), turned to 0 degrees
- moved R29 36.2 mm to (79.5, 117.5), turned to 0 degrees
- moved D6 6.25 mm to (77.0, 105.5), turned to 180 degrees
- moved R26 6.25 mm to (79.5, 105.5), turned to 180 degrees
- moved U11 4.01 mm to (84.5, 63.8)
- moved D11 3.25 mm to (77.0, 102.5)
- moved D7 3.25 mm to (77.0, 111.5)
- moved R27 3.25 mm to (79.5, 111.5)
- moved R31 3.25 mm to (79.5, 102.5)
- moved Q5 2.45 mm to (93.8, 95.2)
- moved R53 2.41 mm to (98.0, 92.0)
- moved C1 2.00 mm to (124.8, 113.5)
- moved C2 2.00 mm to (136.2, 112.8)
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Connections:
- D6 pad 1: Net-(D6-Pad1) -> /XA_5V
- D6 pad 2: GND -> Net-(D6-Pad2)
- IC1 pad 2: /USART1_TX -> /USART2_TX
- IC1 pad 3: /USART1_RX -> /USART2_RX
- P15 pad 3: /USART4_TX -> /USART6_TX
- P15 pad 4: /USART4_RX -> /USART6_RX
- P16 pad 3: /USART3_TX -> /USART1_TX
- P16 pad 4: /USART3_RX -> /USART1_RX
- P8 pad 3: /USART2_TX -> /UART5_TX
- P8 pad 4: /USART2_RX -> /UART5_RX
- P9 pad 3: /UART5_TX -> /USART4_TX
- P9 pad 4: /UART5_RX -> /USART4_RX
- R26 pad 1: Net-(D6-Pad1) -> GND
- R26 pad 2: /XA_5V -> Net-(D6-Pad2)
- U3 pad 5: /USART6_TX -> /USART3_TX
- U3 pad 6: /USART6_RX -> /USART3_RX
Routing:
- net /USART1_RX: track 17.7 -> 80.3 mm
- net /USART1_TX: track 16.1 -> 78.6 mm, vias 0 -> 2
- net /USART6_TX: track 5.13 -> 59.4 mm, vias 0 -> 3
- net /USART6_RX: track 6.07 -> 58.8 mm, vias 0 -> 3
- net /PD1: track 9.71 -> 57.1 mm, vias 1 -> 3
- net /PD3: track 12.6 -> 57.9 mm, vias 1 -> 4
- net /USART3_RX: track 13.0 -> 58.3 mm, vias 1 -> 2
- net /USART3_TX: track 13.5 -> 57.6 mm, vias 1 -> 2
- net /PD4: track 14.1 -> 53.3 mm, vias 1 -> 3
- net /BUS_5V: track 0.00 -> 34.5 mm, vias 0 -> 4
- net /PD0: track 8.79 -> 41.2 mm, vias 0 -> 6
- net +5V: track 353.5 -> 383.0 mm, vias 12 -> 13
- net /USART2_TX: track 69.1 -> 41.8 mm, vias 4 -> 2
- net /USART2_RX: track 71.0 -> 44.5 mm, vias 4 -> 2
- net /NRST: track 122.0 -> 102.4 mm, vias 8 -> 7
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