File: stm32f4-cosmos/stm32f4_cosmos/stm32f4_cosmos.sch (KiCad schematic (older format))
At the start: 191 parts, among them IC1 PIC24FJ64GB004, P1 PICKit3, P10 5V, P11 CAN0, P12 CAN1, P13 CAN0, P14 CAN1, P15 SERIAL, P16 SERIAL, P17 12V, P18 SWD, P2 SBDBT, P23 A/D, P24 PWM, P25 A/D_batt, P26 PWM_batt, P27 EMERGENCY_CHECK, P28 I/O_3.3V, P29 I/O_5V, P3 ENC, P30 I/O_3.3V_batt, P31 I/O_5V_batt, P4 ENC, P5 SERIALx, P6 ENC, P7 ENC, P8 SERIAL, P9 SERIAL, Q1 P_FET, Q2 P_FET, Q3 P_FET, Q4 NPN, Q5 NPN, SW1 POWER_ON, SW2 SW1, SW3 SW0, SW4 SW2, SW5 SW3, U1 STM32F407VG, U10 LOGO, U11 LOGO, U12 25LC010A, U2 AZ1086H, U3 MCP2221A, U4 AP3211, U5 MAX3051, U6 MAX3051, U7 AQM1602_BL, U8 OSTBABS4C2B, U9 LOGO, X1 8MHz

Commit message: 良い感じ.
Parts:
- D18: value CAN_BUS_12V -> 12V
Changed lines of the file:
@@
 U 1 1 5C5AC0ED
 P 3625 13350
-F 0 "D3" H 3625 13565 50  0000 C CNN
-F 1 "SERIALx_RX" H 3625 13474 50  0000 C CNN
+F 0 "D3" H 3625 13175 50  0000 C CNN
+F 1 "SERIALx_RX" H 3625 13250 50  0000 C CNN
 F 2 "LEDs:LED_0603" H 3625 13350 60  0001 C CNN
 F 3 "" H 3625 13350 60  0000 C CNN
 	1    3625 13350
-	1    0    0    -1
+	-1   0    0    1
 $EndComp
 $Comp
@@
 U 1 1 5C5AC173
 P 3625 13625
-F 0 "D4" H 3625 13840 50  0000 C CNN
-F 1 "SERIALx_TX" H 3625 13749 50  0000 C CNN
+F 0 "D4" H 3625 13450 50  0000 C CNN
+F 1 "SERIALx_TX" H 3625 13525 50  0000 C CNN
 F 2 "LEDs:LED_0603" H 3625 13625 60  0001 C CNN
 F 3 "" H 3625 13625 60  0000 C CNN
 	1    3625 13625
-	1    0    0    -1
+	-1   0    0    1
 $EndComp
 $Comp
@@
 U 1 1 5C5AC201
 P 3625 13900
-F 0 "D5" H 3625 14115 50  0000 C CNN
-F 1 "SERIALx_ACTIVE" H 3625 14024 50  0000 C CNN
+F 0 "D5" H 3625 13725 50  0000 C CNN
+F 1 "SERIALx_ACTIVE" H 3625 13800 50  0000 C CNN
 F 2 "LEDs:LED_0603" H 3625 13900 60  0001 C CNN
 F 3 "" H 3625 13900 60  0000 C CNN
 	1    3625 13900
-	1    0    0    -1
-$EndComp
-$Comp
-L power:GND #PWR025
-U 1 1 5C5AC3F0
-P 3850 13925
-F 0 "#PWR025" H 3850 13925 30  0001 C CNN
-F 1 "GND" H 3850 13855 30  0001 C CNN
-F 2 "" H 3850 13925 60  0000 C CNN
-F 3 "" H 3850 13925 60  0000 C CNN
-	1    3850 13925
-	1    0    0    -1
+	-1   0    0    1
 $EndComp
 Wire Wire Line
-	3850 13925 3850 13900
-Wire Wire Line
 	3850 13350 3825 13350
 Wire Wire Line
@@
 Wire Wire Line
 	3850 13900 3825 13900
-Connection ~ 3850 13900
 Wire Wire Line
 	3850 13900 3850 13625
@@
 P 2300 1425
 F 0 "D18" H 2300 1640 50  0000 C CNN
-F 1 "CAN_BUS_12V" H 2300 1549 50  0000 C CNN
+F 1 "12V" H 2300 1549 50  0000 C CNN
 F 2 "LEDs:LED_0603" H 2300 1425 60  0001 C CNN
 F 3 "" H 2300 1425 60  0000 C CNN
@@
 PE8
 Text Label 18175 3700 2    50   ~ 0
-PE8
-Text Label 18175 3300 2    50   ~ 0
 PE7
+Text Label 18175 3300 2    50   ~ 0
+PE8
 Text Label 13650 6150 0    50   ~ 0
 PE10
@@
 Text Label 3650 8050 2    50   ~ 0
 CAN1_RX
-Text Label 19975 5550 0    50   ~ 0
+Text Label 16675 5700 2    50   ~ 0
 PD1
 Text Label 3650 8150 2    50   ~ 0
 CAN1_TX
-Text Label 16275 5675 2    50   ~ 0
+Text Label 19975 5600 0    50   ~ 0
 PD0
 Text Label 20650 5900 2    50   ~ 0
@@
 Text Notes 2450 8100 0    50   ~ 0
 PA12,11 -> can1.
+$Comp
+L power:+3.3V #PWR?
+U 1 1 5C6BBC45
+P 3850 13325
+F 0 "#PWR?" H 3850 13285 30  0001 C CNN
+F 1 "+3.3V" V 3859 13433 30  0000 L CNN
+F 2 "" H 3850 13325 60  0000 C CNN
+F 3 "" H 3850 13325 60  0000 C CNN
+	1    3850 13325
+	1    0    0    -1
+$EndComp
+Wire Wire Line
+	3850 13350 3850 13325
+Connection ~ 3850 13350
 $EndSCHEMATC

Commit message: あと四本.
Parts:
- added U13: LOGO, Mizz_lib:Enc_19.3x7.0_silk, symbol myDevice:LOGO
- U11: footprint Mizz_lib:PPTP_CANT_silk_20x20 -> Mizz_lib:PPTP_uva_silk_20x18
Changed lines of the file:
@@
 $EndComp
 Text Label 21700 13450 0    50   ~ 0
-USART1_TX
+USART2_TX
 NoConn ~ 21700 13750
 NoConn ~ 21700 13650
@@
 	3850 13900 3850 13625
 Text Label 21700 13550 0    50   ~ 0
-USART1_RX
+USART2_RX
 Text Label 13650 7150 0    50   ~ 0
 UART5_RX
@@
 L device:R R26
 U 1 1 5C7AE1A7
-P 1950 1750
-F 0 "R26" V 1758 1750 40  0000 C CNN
-F 1 "510" V 1834 1750 40  0000 C CNN
-F 2 "Resistors_SMD:R_0603" V 1880 1750 30  0001 C CNN
-F 3 "" H 1950 1750 30  0000 C CNN
-	1    1950 1750
+P 2350 1750
+F 0 "R26" V 2158 1750 40  0000 C CNN
+F 1 "510" V 2234 1750 40  0000 C CNN
+F 2 "Resistors_SMD:R_0603" V 2280 1750 30  0001 C CNN
+F 3 "" H 2350 1750 30  0000 C CNN
+	1    2350 1750
 	0    1    1    0
 $EndComp
@@
 L device:LED D6
 U 1 1 5C7AE444
-P 2300 1750
-F 0 "D6" H 2300 1965 50  0000 C CNN
-F 1 "SELF_5V" H 2300 1874 50  0000 C CNN
-F 2 "LEDs:LED_0603" H 2300 1750 60  0001 C CNN
-F 3 "" H 2300 1750 60  0000 C CNN
-	1    2300 1750
+P 2000 1750
+F 0 "D6" H 2000 1965 50  0000 C CNN
+F 1 "SELF_5V" H 2000 1874 50  0000 C CNN
+F 2 "LEDs:LED_0603" H 2000 1750 60  0001 C CNN
+F 3 "" H 2000 1750 60  0000 C CNN
+	1    2000 1750
 	1    0    0    -1
 $EndComp
@@
 F 0 "U11" H 22378 1253 60  0000 L CNN
 F 1 "LOGO" H 22378 1147 60  0000 L CNN
-F 2 "Mizz_lib:PPTP_CANT_silk_20x20" H 22100 1200 60  0001 C CNN
+F 2 "Mizz_lib:PPTP_uva_silk_20x18" H 22100 1200 60  0001 C CNN
 F 3 "" H 22100 1200 60  0000 C CNN
 	1    22100 1200
@@
 Text Label 15925 3750 2    50   ~ 0
 PB11
-Text Label 4200 14700 2    50   ~ 0
-UART5_RX
-Text Label 3150 14600 2    50   ~ 0
-USART2_TX
 Text Label 3150 14700 2    50   ~ 0
-USART2_RX
+UART5_RX
 Text Label 4200 15275 2    50   ~ 0
-USART3_TX
+USART1_TX
 Text Label 4200 15375 2    50   ~ 0
-USART3_RX
+USART1_RX
 Text Label 1550 13600 2    50   ~ 0
-USART6_TX
+USART3_TX
 Text Label 1550 13675 2    50   ~ 0
-USART6_RX
+USART3_RX
 Text Label 3150 15275 2    50   ~ 0
-USART4_TX
+USART6_TX
 Text Label 3150 15375 2    50   ~ 0
-USART4_RX
+USART6_RX
 Text Label 4200 14600 2    50   ~ 0
+USART4_TX
+Text Label 4200 14700 2    50   ~ 0
+USART4_RX
+Text Label 3150 14600 2    50   ~ 0
 UART5_TX
 $Sheet
@@
 PA12,11 -> can1.
 $Comp
-L power:+3.3V #PWR?
+L power:+3.3V #PWR0150
 U 1 1 5C6BBC45
 P 3850 13325
-F 0 "#PWR?" H 3850 13285 30  0001 C CNN
+F 0 "#PWR0150" H 3850 13285 30  0001 C CNN
 F 1 "+3.3V" V 3859 13433 30  0000 L CNN
 F 2 "" H 3850 13325 60  0000 C CNN
@@
 	3850 13350 3850 13325
 Connection ~ 3850 13350
+$Comp
+L myDevice:LOGO U13
+U 1 1 5C5FBB63
+P 19550 1200
+F 0 "U13" H 19828 1253 60  0000 L CNN
+F 1 "LOGO" H 19828 1147 60  0000 L CNN
+F 2 "Mizz_lib:Enc_19.3x7.0_silk" H 19550 1200 60  0001 C CNN
+F 3 "" H 19550 1200 60  0000 C CNN
+	1    19550 1200
+	1    0    0    -1
+$EndComp
 $EndSCHEMATC
