File: Parent_Turtle_RC19ver6.kagoshima_link_main_ver/Parent_Turtle_RC19main.kicad_pcb (KiCad board)
At the start: 2 copper layers, 70 x 60 mm, 90 parts, among them P1 CONN_02X15, P10 WRITING, P11 ADC, P12 5V_in, P13 ADC/Vdd/GND, P14 PWM, P17 SERIAL0, P18 ENC2, P19 ENC3, P2 CONN_02X15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

Commit message: kagoshima_link_main.
Routing:
- net /GP3: track 16.2 -> 15.2 mm
Changed lines of the file:
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@@
     (thickness 1.6)
     (drawings 13)
-    (tracks 578)
+    (tracks 576)
     (zones 0)
     (modules 90)
@@
   (segment (start 135.08 109.22) (end 135.08 111.14) (width 0.3) (layer B.Cu) (net 103))
   (segment (start 135.08 111.14) (end 136.03 112.09) (width 0.3) (layer B.Cu) (net 103))
-  (segment (start 131.53 118.675) (end 132.02 119.165) (width 0.3) (layer B.Cu) (net 103))
   (segment (start 135.51 117.78) (end 136.03 117.26) (width 0.3) (layer B.Cu) (net 103))
   (segment (start 135.51 117.785) (end 135.51 117.78) (width 0.3) (layer B.Cu) (net 103))
@@
   (segment (start 131.95 118.755) (end 132.36 119.165) (width 0.3) (layer B.Cu) (net 103))
   (segment (start 131.95 117.4) (end 131.95 118.755) (width 0.3) (layer B.Cu) (net 103))
-  (segment (start 132.36 119.165) (end 132.02 119.165) (width 0.3) (layer B.Cu) (net 103))
   (segment (start 134.13 119.165) (end 135.51 117.785) (width 0.3) (layer B.Cu) (net 103))
   (segment (start 132.36 119.165) (end 134.13 119.165) (width 0.3) (layer B.Cu) (net 103))
