File: Parent_Turtle_RC19ver6.kagoshima_link_main_ver/Parent_Turtle_RC19main.sch (KiCad schematic (older format))
At the start: 90 parts, among them P1 CONN_02X15, P10 WRITING, P11 ADC, P12 5V_in, P13 ADC/Vdd/GND, P14 PWM, P17 SERIAL0, P18 ENC2, P19 ENC3, P2 CONN_02X15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

Commit message: kagoshima link main.
Parts:
- removed D1: LED, LEDs:LED-3MM, symbol device:LED
Changed lines of the file:
@@
-$EndComp
-$Comp
-L device:LED D1
-U 1 1 5B3F32F5
-P 6900 1250
-F 0 "D1" H 6900 1350 50  0000 C CNN
-F 1 "LED" H 6900 1150 50  0000 C CNN
-F 2 "LEDs:LED-3MM" H 6900 1250 60  0001 C CNN
-F 3 "" H 6900 1250 60  0000 C CNN
-	1    6900 1250
-	-1   0    0    1
 $EndComp
 $Comp

Commit message: RC19 mains.
Parts:
- added D1: LED, LEDs:LED-3MM, symbol device:LED
Changed lines of the file:
@@
 Text Label 3150 3950 2    60   ~ 0
 E14
+$Comp
+L device:LED D1
+U 1 1 5C7D6976
+P 6900 1250
+F 0 "D1" H 6900 1350 50  0000 C CNN
+F 1 "LED" H 6900 1150 50  0000 C CNN
+F 2 "LEDs:LED-3MM" H 6900 1250 60  0001 C CNN
+F 3 "" H 6900 1250 60  0000 C CNN
+	1    6900 1250
+	-1   0    0    1
+$EndComp
 $EndSCHEMATC
