File: stm32f4_Centaurus/stm32f4_Centaurus/stm32f4_Centaurus.kicad_pcb (KiCad board)
At the start: 2 copper layers, 100 x 94 mm, 192 parts, among them IC1 PIC24FJ64GB004, P1 PICKit3, P10 5V, P11 CAN0, P12 CAN1, P13 CAN0, P14 CAN1, P15 SERIAL, P16 SERIAL, P17 12V, P18 SWD, P2 SBDBT, P23 A/D, P24 PWM, P25 A/D_batt, P26 PWM_batt, P27 EMERGENCY_CHECK, P28 I/O_3.3V, P29 I/O_5V, P3 ENC, P30 I/O_3.3V_batt, P31 I/O_5V_batt, P4 ENC, P5 SERIALx, P6 ENC, P7 ENC, P8 SERIAL, P9 SERIAL, Q1 P_FET, Q2 P_FET, Q3 P_FET, Q4 NPN, Q5 NPN, SW1 POWER_ON, SW2 SW1, SW3 SW0, SW4 SW2, SW5 SW3, U1 STM32F407VG, U10 LOGO, U11 LOGO, U12 25LC010A, U13 LOGO, U2 AZ1086H, U3 MCP2221A, U4 AP3211, U5 MAX3051, U6 MAX3051, U7 AQM1602_BL, U8 OSTBABS4C2B, U9 LOGO, X1 8MHz

Commit message: cosmos -> Centaurus, 加工データの追加.
Parts:
- D3: value SERIALx_RX -> SERIAL1_RX
- D4: value SERIALx_TX -> SERIAL1_TX
- D5: value SERIALx_ACTIVE -> SERIAL1_ACTIVE
- P15: value SERIAL -> SERIAL2
- P16: value SERIAL -> SERIAL0
- P2: value SBDBT -> SERIAL5(SBDBT)
- P3: value ENC -> ENC1
- P4: value ENC -> ENC2
- P5: value SERIALx -> SERIAL1
- P6: value ENC -> ENC3
- P7: value ENC -> ENC0
- P8: value SERIAL -> SERIAL4
- P9: value SERIAL -> SERIAL3
- moved R63 14.2 mm to (104.5, 89.2), turned to 90 degrees
- moved R62 12.3 mm to (116.0, 71.2)
- moved C21 1.90 mm to (81.6, 111.5), turned to 90 degrees
- moved R13 1.75 mm to (146.2, 76.0)
- moved R14 1.75 mm to (146.2, 77.8)
- moved R18 1.75 mm to (146.2, 79.7)
- moved R20 1.75 mm to (146.2, 74.2)
- moved C14 1.50 mm to (151.5, 71.8)
- moved P6 1.50 mm to (149.5, 78.0)
- moved U10 1.14 mm to (59.8, 68.8)
- moved R6 1.06 mm to (146.4, 88.4)
- moved R11 1.06 mm to (146.4, 86.7)
- moved R7 1.06 mm to (146.4, 90.2)
- moved R9 1.06 mm to (146.4, 92.0)
- moved C16 1.00 mm to (127.5, 136.8)
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Routing:
- net /UART5_TX: track 13.7 -> 70.4 mm, vias 1 -> 6
- net /UART5_RX: track 15.6 -> 71.4 mm, vias 1 -> 7
- net /USART4_TX: track 14.6 -> 67.3 mm, vias 1 -> 4
- net /USART4_RX: track 24.0 -> 68.9 mm, vias 2 -> 5
- net /SPI2_SCK: track 27.0 -> 11.3 mm
- net Net-(R63-Pad2): track 1.92 -> 16.0 mm
- net /SPI2_MISO: track 21.5 -> 8.01 mm
- net Net-(R62-Pad1): track 1.99 -> 14.8 mm, vias 0 -> 2
- net +5V: track 383.0 -> 373.9 mm
- net /CAN_BUS_5V: track 4.58 -> 13.1 mm, vias 0 -> 1
- net GND: track 7.26 -> 15.4 mm, vias 59 -> 65
- net +3.3V: track 475.3 -> 470.6 mm, vias 29 -> 31
- net /PD4: track 53.3 -> 55.7 mm, vias 3 -> 4
- net /PD7: track 57.6 -> 59.6 mm
- net /PD3: track 57.9 -> 56.2 mm
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Other:
- board size 100 x 94 mm -> 100 x 95 mm
- board text added: "100x95"
- board text added: "3"
- board text added: "9"
- board text added: "Desgined by A.Mizuta in 2019/02/08. Special Thanks : Y.Shoda, T.Yamada."
- board text added: "STM32F407VGT6 Board "Centaurus" ver.1.0."
- board text removed: "100x100"
- board text removed: "Desgined by A.Mizuta in 2019/02/05. Special Thanks : Y.Shoda, T.Yamada."
- board text removed: "STM32F407VGT6 Board "" ver.1.0."

Commit message: Add MR2 main circuit project.
Parts:
- added D29: DIODE, Mizz_lib:SOD-123, B.Cu at (80.3, 104.3)
- P2: value SERIAL5(SBDBT) -> SERIAL5_SBDBT
- SW1: footprint Mizz_lib:2MS1-T1-B4-VS2-Q-E -> Buttons_Switches_ThroughHole:SW_Micro_SPST
- moved C11 5.72 mm to (122.2, 66.8)
- moved C13 5.72 mm to (125.8, 66.8)
Connections:
- C19 pad 1: +12V -> Net-(C19-Pad1)
- U4 pad 4: +12V -> Net-(C19-Pad1)
- U4 pad 5: +12V -> Net-(C19-Pad1)
Routing:
- net +12V: track 102.2 -> 92.7 mm, vias 1 -> 2
- net Net-(C19-Pad1): track 0.00 -> 6.77 mm
- net /OSC_IN: track 9.04 -> 12.5 mm
- net /OSC_OUT: track 8.42 -> 11.7 mm
- net (no net): track 2.44 -> 0.00 mm, vias 7 -> 5
- net Net-(D15-Pad1): track 13.9 -> 12.7 mm
- net /NRST: track 103.2 -> 102.1 mm
- net GND: vias 65 -> 64

Commit message: 一応完成.
Parts:
- removed C31, C32: 0.1u, Capacitors_SMD:C_0603
- added D30: DIODE, Mizz_lib:SOD-123, B.Cu at (70.0, 86.8)
- added D31: DIODE, Mizz_lib:SOD-123, B.Cu at (75.8, 87.2)
- added D32: DIODE, Mizz_lib:SOD-123, B.Cu at (68.2, 83.5)
- added D33: DIODE, Mizz_lib:SOD-123, B.Cu at (63.0, 96.0)
- added D34: DIODE, Mizz_lib:SOD-123, B.Cu at (68.2, 96.0)
- added D35: XA4_12V, LEDs:LED_0603, F.Cu at (68.5, 81.0)
- added D36: CAN0_BUS, Mizz_lib:LED_0603, F.Cu at (67.5, 92.2)
- added D37: CAN1_BUS, Mizz_lib:LED_0603, F.Cu at (67.5, 94.0)
- added D38: DIODE, Mizz_lib:SOD-123, B.Cu at (59.8, 96.8)
- added D39: DIODE, Mizz_lib:SOD-123, B.Cu at (66.0, 108.8)
- added Q6: P_FET, TO_SOT_Packages_SMD:SOT-23, B.Cu at (72.8, 86.5)
- added R65: 10k, Resistors_SMD:R_0603, B.Cu at (72.8, 83.8)
- added R66: 1.2k, Resistors_SMD:R_0603, B.Cu at (70.2, 81.0)
- added R67: 1.2k, Resistors_SMD:R_0603, B.Cu at (63.0, 92.2)
- added R68: 1.2k, Resistors_SMD:R_0603, B.Cu at (63.0, 94.0)
- C22, C23: value 0.1u -> 1u
- D8: value CAN_BUS_5V -> 12V_to_5V
- moved C22 2.50 mm to (64.5, 99.8)
- moved C23 2.50 mm to (64.5, 112.8)
- moved JP2 2.20 mm to (55.0, 123.5)
- moved JP1 2.20 mm to (55.0, 94.0)
- moved P17 0.70 mm to (66.2, 125.5)
- moved R50 0.25 mm to (79.5, 80.8)
- moved R52 0.15 mm to (82.0, 80.8)
Connections:
- C22 pad 2: +12V -> CAN0_BUS_Vdd
- C23 pad 2: +12V -> CAN1_BUS_Vdd
- C42 pad 2: +12V -> XA4_12V
- C5 pad 1: /CAN_BUS_5V -> /12V_TO_5V
- D15 pad 2: /CAN_BUS_5V -> /12V_TO_5V
- P11 pad 2: +12V -> CAN0_BUS_Vdd
- P12 pad 2: +12V -> CAN1_BUS_Vdd
- P13 pad 2: +12V -> CAN0_BUS_Vdd
- P14 pad 2: +12V -> CAN1_BUS_Vdd
- P27 pad 2: +12V -> XA4_12V
- R28 pad 2: /CAN_BUS_5V -> /12V_TO_5V
Routing:
- net +12V: track 92.7 -> 60.9 mm
- net /CAN_BUS_12V: track 0.00 -> 17.1 mm, vias 0 -> 4
- net /CAN1_BUS_12V: track 0.00 -> 15.0 mm, vias 0 -> 2
- net /CAN_BUS_5V: track 13.1 -> 0.00 mm, vias 1 -> 0
- net CAN1_BUS_Vdd: track 0.00 -> 12.1 mm
- net CAN0_BUS_Vdd: track 0.00 -> 11.6 mm
- net /12V_TO_5V: track 0.00 -> 11.3 mm, vias 0 -> 1
- net /XA4-12V: track 0.00 -> 8.52 mm
- net /CAN0_BUS_12V: track 0.00 -> 6.64 mm, vias 0 -> 1
- net XA4_12V: track 0.00 -> 5.03 mm
- net Net-(D37-Pad1): track 0.00 -> 4.40 mm, vias 0 -> 1
- net Net-(D36-Pad1): track 0.00 -> 2.84 mm, vias 0 -> 1
- net Net-(D31-Pad2): track 0.00 -> 2.10 mm
- net Net-(JP2-Pad1): track 6.68 -> 7.75 mm
- net /CAN0_L: track 30.9 -> 31.7 mm
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