File: stm32f4_Centaurus/stm32f4_Centaurus/stm32f4_Centaurus.sch (KiCad schematic (older format))
At the start: 192 parts, among them IC1 PIC24FJ64GB004, P1 PICKit3, P10 5V, P11 CAN0, P12 CAN1, P13 CAN0, P14 CAN1, P15 SERIAL, P16 SERIAL, P17 12V, P18 SWD, P2 SBDBT, P23 A/D, P24 PWM, P25 A/D_batt, P26 PWM_batt, P27 EMERGENCY_CHECK, P28 I/O_3.3V, P29 I/O_5V, P3 ENC, P30 I/O_3.3V_batt, P31 I/O_5V_batt, P4 ENC, P5 SERIALx, P6 ENC, P7 ENC, P8 SERIAL, P9 SERIAL, Q1 P_FET, Q2 P_FET, Q3 P_FET, Q4 NPN, Q5 NPN, SW1 POWER_ON, SW2 SW1, SW3 SW0, SW4 SW2, SW5 SW3, U1 STM32F407VG, U10 LOGO, U11 LOGO, U12 25LC010A, U13 LOGO, U2 AZ1086H, U3 MCP2221A, U4 AP3211, U5 MAX3051, U6 MAX3051, U7 AQM1602_BL, U8 OSTBABS4C2B, U9 LOGO, X1 8MHz

Commit message: cosmos -> Centaurus, 加工データの追加.
Parts:
- D3: value SERIALx_RX -> SERIAL1_RX
- D4: value SERIALx_TX -> SERIAL1_TX
- D5: value SERIALx_ACTIVE -> SERIAL1_ACTIVE
- P15: value SERIAL -> SERIAL2
- P16: value SERIAL -> SERIAL0
- P2: value SBDBT -> SERIAL5(SBDBT)
- P3: value ENC -> ENC1
- P4: value ENC -> ENC2
- P5: value SERIALx -> SERIAL1
- P6: value ENC -> ENC3
- P7: value ENC -> ENC0
- P8: value SERIAL -> SERIAL4
- P9: value SERIAL -> SERIAL3
Changed lines of the file:
@@
 P 22000 10450
 F 0 "P2" H 22026 10775 50  0000 C CNN
-F 1 "SBDBT" H 22026 10684 50  0000 C CNN
+F 1 "SERIAL5(SBDBT)" H 22026 10684 50  0000 C CNN
 F 2 "Mizz_lib:USB_A" V 21950 10350 50  0001 C CNN
 F 3 "" V 21950 10350 50  0000 C CNN
@@
 P 2000 14450
 F 0 "P5" H 2076 14775 50  0000 C CNN
-F 1 "SERIALx" H 2076 14684 50  0000 C CNN
+F 1 "SERIAL1" H 2076 14684 50  0000 C CNN
 F 2 "Connect:USB_Micro-B" V 1950 14350 50  0001 C CNN
 F 3 "" V 1950 14350 50  0000 C CNN
@@
 P 3350 14550
 F 0 "P8" H 3428 14591 50  0000 L CNN
-F 1 "SERIAL" H 3428 14500 50  0000 L CNN
+F 1 "SERIAL4" H 3428 14500 50  0000 L CNN
 F 2 "RP_KiCAD_Connector:XA_4T" H 3350 14550 50  0001 C CNN
 F 3 "" H 3350 14550 50  0000 C CNN
@@
 P 4400 14550
 F 0 "P9" H 4478 14591 50  0000 L CNN
-F 1 "SERIAL" H 4478 14500 50  0000 L CNN
+F 1 "SERIAL3" H 4478 14500 50  0000 L CNN
 F 2 "RP_KiCAD_Connector:XA_4T" H 4400 14550 50  0001 C CNN
 F 3 "" H 4400 14550 50  0000 C CNN
@@
 P 3625 13350
 F 0 "D3" H 3625 13175 50  0000 C CNN
-F 1 "SERIALx_RX" H 3625 13250 50  0000 C CNN
+F 1 "SERIAL1_RX" H 3625 13250 50  0000 C CNN
 F 2 "LEDs:LED_0603" H 3625 13350 60  0001 C CNN
 F 3 "" H 3625 13350 60  0000 C CNN
@@
 P 3625 13625
 F 0 "D4" H 3625 13450 50  0000 C CNN
-F 1 "SERIALx_TX" H 3625 13525 50  0000 C CNN
+F 1 "SERIAL1_TX" H 3625 13525 50  0000 C CNN
 F 2 "LEDs:LED_0603" H 3625 13625 60  0001 C CNN
 F 3 "" H 3625 13625 60  0000 C CNN
@@
 P 3625 13900
 F 0 "D5" H 3625 13725 50  0000 C CNN
-F 1 "SERIALx_ACTIVE" H 3625 13800 50  0000 C CNN
+F 1 "SERIAL1_ACTIVE" H 3625 13800 50  0000 C CNN
 F 2 "LEDs:LED_0603" H 3625 13900 60  0001 C CNN
 F 3 "" H 3625 13900 60  0000 C CNN
@@
 P 12150 13850
 F 0 "P3" H 12227 13891 50  0000 L CNN
-F 1 "ENC" H 12227 13800 50  0000 L CNN
+F 1 "ENC1" H 12227 13800 50  0000 L CNN
 F 2 "RP_KiCAD_Connector:XA_4T" H 12150 13850 50  0001 C CNN
 F 3 "" H 12150 13850 50  0000 C CNN
@@
 P 13450 13850
 F 0 "P6" H 13527 13891 50  0000 L CNN
-F 1 "ENC" H 13527 13800 50  0000 L CNN
+F 1 "ENC3" H 13527 13800 50  0000 L CNN
 F 2 "RP_KiCAD_Connector:XA_4T" H 13450 13850 50  0001 C CNN
 F 3 "" H 13450 13850 50  0000 C CNN
@@
 P 12150 14875
 F 0 "P4" H 12227 14916 50  0000 L CNN
-F 1 "ENC" H 12227 14825 50  0000 L CNN
+F 1 "ENC2" H 12227 14825 50  0000 L CNN
 F 2 "RP_KiCAD_Connector:XA_4T" H 12150 14875 50  0001 C CNN
 F 3 "" H 12150 14875 50  0000 C CNN
@@
 P 13450 14875
 F 0 "P7" H 13527 14916 50  0000 L CNN
-F 1 "ENC" H 13527 14825 50  0000 L CNN
+F 1 "ENC0" H 13527 14825 50  0000 L CNN
 F 2 "RP_KiCAD_Connector:XA_4T" H 13450 14875 50  0001 C CNN
 F 3 "" H 13450 14875 50  0000 C CNN
@@
 P 3350 15225
 F 0 "P15" H 3428 15266 50  0000 L CNN
-F 1 "SERIAL" H 3428 15175 50  0000 L CNN
+F 1 "SERIAL2" H 3428 15175 50  0000 L CNN
 F 2 "RP_KiCAD_Connector:XA_4T" H 3350 15225 50  0001 C CNN
 F 3 "" H 3350 15225 50  0000 C CNN
@@
 P 4400 15225
 F 0 "P16" H 4478 15266 50  0000 L CNN
-F 1 "SERIAL" H 4478 15175 50  0000 L CNN
+F 1 "SERIAL0" H 4478 15175 50  0000 L CNN
 F 2 "RP_KiCAD_Connector:XA_4T" H 4400 15225 50  0001 C CNN
 F 3 "" H 4400 15225 50  0000 C CNN

Commit message: Add MR2 main circuit project.
Parts:
- added D29, D? (x3): DIODE, Mizz_lib:SOD-123, symbol device:DIODE
- added D? (x4): DIODE, symbol device:DIODE
- added D? (x2): LED, symbol device:LED
- added D?: XA_12V, LEDs:LED_0603, symbol device:LED
- added Q?: P_FET, TO_SOT_Packages_SMD:SOT-23, symbol Miz:MOSFET_P
- added R? (x2): 1.2k, symbol device:R
- added R?: 1.2k, Resistors_SMD:R_0603, symbol device:R
- added R?: R, symbol device:R
- D8: value CAN_BUS_5V -> 12V_to_5V
- P2: value SERIAL5(SBDBT) -> SERIAL5_SBDBT
- SW1: footprint Mizz_lib:2MS1-T1-B4-VS2-Q-E -> Buttons_Switches_ThroughHole:SW_Micro_SPST
Connections:
- net labels added: 12V_TO_5V, CAN0_BUS_12V, CAN0_BUS_Vdd, CAN1_BUS_12V, CAN1_BUS_Vdd, CAN_BUS_12V, XA4_12V, XA_12V
- wire segments 397 -> 414
Other:
- moved on the sheet: C18, C19, C20, C21, C22, C23, C31, C32, C5, C6, C7, JP1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

Commit message: 一応完成.
Parts:
- removed C31, C32: 0.1u, Capacitors_SMD:C_0603, symbol device:C
- C22, C23: value 0.1u -> 1u
- D33, D34, D38, D39: renamed from D?; footprint (none) -> Mizz_lib:SOD-123
- D35: renamed from D?; value XA_12V -> XA4_12V
- D36: renamed from D?; value LED -> CAN0_BUS; footprint (none) -> Mizz_lib:LED_0603
- D37: renamed from D?; value LED -> CAN1_BUS; footprint (none) -> Mizz_lib:LED_0603
- R65: renamed from R?; value R -> 10k; footprint (none) -> Resistors_SMD:R_0603
- R67, R68: renamed from R?; footprint (none) -> Resistors_SMD:R_0603
- gave numbers to parts that had none: 5
Connections:
- net labels added: XA4-12V
- net labels removed: XA_12V
- wire segments 414 -> 406
Other:
- moved on the sheet: C20, C21, C22, C23, D36, D37, JP1, JP2, P11, P12, P13, P14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

Commit message: ver.0とver.1の両方をあげておく.
Changed lines of the file:
@@
 $Descr A2 23386 16535
 encoding utf-8
-Sheet 1 10
+Sheet 1 9
 Title ""
 Date ""
@@
 	-1   0    0    1
 $EndComp
+$Sheet
+S 17250 7250 5450 2025
+U 5C7DEB05
+F0 "CAN" 50
+F1 "CAN.sch" 50
+$EndSheet
 $EndSCHEMATC

Commit message: これはくそ基板.
Parts:
- D12, D13, D14, D15, D16, D17, D20, D26, D27, D28, D29, D30, D31, D32, D33, D34, D38, D39: symbol device:DIODE -> stm32f4_Centaurus-rescue:DIODE-device
- Q4, Q5: symbol device:NPN -> stm32f4_Centaurus-rescue:NPN-device
- U10, U11, U13, U9: symbol myDevice:LOGO -> stm32f4_Centaurus-rescue:LOGO-myDevice
- U5, U6: symbol myDevice:MAX3051 -> stm32f4_Centaurus-rescue:MAX3051-myDevice
- U7: symbol Miz:AQM1602_BL -> stm32f4_Centaurus-rescue:AQM1602_BL-Miz
- U8: symbol myDevice:OSTBABS4C2B -> stm32f4_Centaurus-rescue:OSTBABS4C2B-myDevice
Changed lines of the file:
@@
 $Descr A2 23386 16535
 encoding utf-8
-Sheet 1 9
+Sheet 1 10
 Title ""
 Date ""
@@
 	6425 2175 6425 2200
 $Comp
-L myDevice:MAX3051 U5
+L stm32f4_Centaurus-rescue:MAX3051-myDevice U5
 U 1 1 5C55F62D
 P 18200 7825
@@
 $EndComp
 $Comp
-L myDevice:MAX3051 U6
+L stm32f4_Centaurus-rescue:MAX3051-myDevice U6
 U 1 1 5C55F6F9
 P 18200 8775
@@
 $EndComp
 $Comp
-L device:DIODE D12
+L stm32f4_Centaurus-rescue:DIODE-device D12
 U 1 1 5C57D240
 P 3700 2600
@@
 $EndComp
 $Comp
-L device:DIODE D13
+L stm32f4_Centaurus-rescue:DIODE-device D13
 U 1 1 5C57D2CD
 P 3875 3425
@@
 Connection ~ 6450 3150
 $Comp
-L device:DIODE D14
+L stm32f4_Centaurus-rescue:DIODE-device D14
 U 1 1 5C69879B
 P 6100 2425
@@
 $EndComp
 $Comp
-L device:DIODE D15
+L stm32f4_Centaurus-rescue:DIODE-device D15
 U 1 1 5C6CB8CA
 P 6675 2825
@@
 $EndComp
 $Comp
-L device:DIODE D17
+L stm32f4_Centaurus-rescue:DIODE-device D17
 U 1 1 5C76574D
 P 7975 3275
@@
 5V
 $Comp
-L device:DIODE D16
+L stm32f4_Centaurus-rescue:DIODE-device D16
 U 1 1 5C7974B6
 P 7775 2475
@@
 Connection ~ 4175 15075
 $Comp
-L Miz:AQM1602_BL U7
+L stm32f4_Centaurus-rescue:AQM1602_BL-Miz U7
 U 1 1 5C850363
 P 21700 5100
@@
 $EndComp
 $Comp
-L device:NPN Q4
+L stm32f4_Centaurus-rescue:NPN-device Q4
 U 1 1 5C850AC4
 P 21150 5900
@@
 	18200 5600 18200 5625
 $Comp
-L myDevice:OSTBABS4C2B U8
+L stm32f4_Centaurus-rescue:OSTBABS4C2B-myDevice U8
 U 1 1 5C9A05DA
 P 18725 4775
@@
 $EndComp
 $Comp
-L device:NPN Q5
+L stm32f4_Centaurus-rescue:NPN-device Q5
 U 1 1 5D035423
 P 20825 3700
@@
 $EndComp
 $Comp
-L device:DIODE D20
+L stm32f4_Centaurus-rescue:DIODE-device D20
 U 1 1 5D0368B7
 P 21125 3300
@@
 NRST
 $Comp
-L myDevice:LOGO U11
+L stm32f4_Centaurus-rescue:LOGO-myDevice U11
 U 1 1 5DCAD440
 P 22100 1200
@@
 $EndComp
 $Comp
-L myDevice:LOGO U10
+L stm32f4_Centaurus-rescue:LOGO-myDevice U10
 U 1 1 5DCADB10
 P 21250 1200
@@
 $EndComp
 $Comp
-L myDevice:LOGO U9
+L stm32f4_Centaurus-rescue:LOGO-myDevice U9
 U 1 1 5DCAEEAA
 P 20400 1200
@@
 Connection ~ 15900 3450
 $Comp
-L device:DIODE D26
+L stm32f4_Centaurus-rescue:DIODE-device D26
 U 1 1 5E6CB6C3
 P 15725 3650
@@
 $EndComp
 $Comp
-L device:DIODE D27
+L stm32f4_Centaurus-rescue:DIODE-device D27
 U 1 1 5E6CC486
 P 17125 3425
@@
 $EndComp
 $Comp
-L device:DIODE D28
+L stm32f4_Centaurus-rescue:DIODE-device D28
 U 1 1 5E6CC877
 P 17125 3825
@@
 Connection ~ 3850 13350
 $Comp
-L myDevice:LOGO U13
+L stm32f4_Centaurus-rescue:LOGO-myDevice U13
 U 1 1 5C5FBB63
 P 19550 1200
@@
 $EndComp
 $Comp
-L device:DIODE D29
+L stm32f4_Centaurus-rescue:DIODE-device D29
 U 1 1 5C73222C
 P 6125 3025
@@
 CAN0_BUS_Vdd
 $Comp
-L device:DIODE D38
+L stm32f4_Centaurus-rescue:DIODE-device D38
 U 1 1 5C7DBE40
 P 21875 8175
@@
 CAN1_BUS_Vdd
 $Comp
-L device:DIODE D39
+L stm32f4_Centaurus-rescue:DIODE-device D39
 U 1 1 5C8C2D01
 P 21875 9125
@@
 12V_TO_5V
 $Comp
-L device:DIODE D30
+L stm32f4_Centaurus-rescue:DIODE-device D30
 U 1 1 5CA9A6E5
 P 9475 2475
@@
 $EndComp
 $Comp
-L device:DIODE D32
+L stm32f4_Centaurus-rescue:DIODE-device D32
 U 1 1 5CA9F856
 P 15675 4100
@@
 $EndComp
 $Comp
-L device:DIODE D31
+L stm32f4_Centaurus-rescue:DIODE-device D31
 U 1 1 5CAD144A
 P 9675 3275
@@
 CAN0_BUS_12V
 $Comp
-L device:DIODE D34
+L stm32f4_Centaurus-rescue:DIODE-device D34
 U 1 1 5CBEF4C3
 P 16000 7800
@@
 CAN1_BUS_12V
 $Comp
-L device:DIODE D33
+L stm32f4_Centaurus-rescue:DIODE-device D33
 U 1 1 5CBEFD4B
 P 16000 7500
