File: stm32f4_Centaurus_ver.1.0/stm32f4_Centaurus/stm32f4_Centaurus.sch (KiCad schematic (older format))
At the start: 207 parts, among them IC1 PIC24FJ64GB004, P1 PICKit3, P10 5V, P11 CAN0, P12 CAN1, P13 CAN0, P14 CAN1, P15 SERIAL2, P16 SERIAL0, P17 12V, P18 SWD, P2 SERIAL5_SBDBT, P23 A/D, P24 PWM, P25 A/D_batt, P26 PWM_batt, P27 EMERGENCY_CHECK, P28 I/O_3.3V, P29 I/O_5V, P3 ENC1, P30 I/O_3.3V_batt, P31 I/O_5V_batt, P4 ENC2, P5 SERIAL1, P6 ENC3, P7 ENC0, P8 SERIAL4, P9 SERIAL3, Q1 P_FET, Q2 P_FET, Q3 P_FET, Q4 NPN, Q5 NPN, Q6 P_FET, SW1 POWER_ON, SW2 SW1, SW3 SW0, SW4 SW2, SW5 SW3, U1 STM32F407VG, U10 LOGO, U11 LOGO, U12 25LC010A, U13 LOGO, U2 AZ1086H, U3 MCP2221A, U4 AP3211, U5 MAX3051, U6 MAX3051, U7 AQM1602_BL, U8 OSTBABS4C2B, U9 LOGO, X1 8MHz

Commit message: ver.0とver.1の両方をあげておく.
Connections:
- net labels added: UART4_RX, UART4_TX
- net labels removed: USART4_RX, USART4_TX
Changed lines of the file:
@@
 UART5_TX
 Text Label 13650 9850 0    50   ~ 0
-USART4_RX
+UART4_RX
 Text Label 13650 9750 0    50   ~ 0
-USART4_TX
+UART4_TX
 Text Label 13650 7850 0    50   ~ 0
 USART3_RX
@@
 USART6_RX
 Text Label 4200 14600 2    50   ~ 0
-USART4_TX
+UART4_TX
 Text Label 4200 14700 2    50   ~ 0
-USART4_RX
+UART4_RX
 Text Label 3150 14600 2    50   ~ 0
 UART5_TX

Commit message: RC19 mains.
Parts:
- removed D10: USE_5V, LEDs:LED_0603, symbol device:LED
- removed D11: 3.3V, LEDs:LED_0603, symbol device:LED
- removed D13, D16, D17, D27, D28, D30, D31, D33, D34: DIODE, Mizz_lib:SOD-123, symbol device:DIODE
- removed D6: SELF_5V, LEDs:LED_0603, symbol device:LED
- removed D7: BUS_5V, LEDs:LED_0603, symbol device:LED
- removed D8: 12V_to_5V, LEDs:LED_0603, symbol device:LED
- removed D9: SW_5V, LEDs:LED_0603, symbol device:LED
- removed Q1, Q2, Q3, Q6: P_FET, TO_SOT_Packages_SMD:SOT-23, symbol Miz:MOSFET_P
- added D10, D11, D6, D7, D8, D9: DIODE, Mizz_lib:SOD-123, symbol device:DIODE
- added D13: XA2_12V, Mizz_lib:LED_0603, symbol device:LED
- added D16: XA_5V, Mizz_lib:LED_0603, symbol device:LED
- added D17: 12V_to_5V, Mizz_lib:LED_0603, symbol device:LED
- added D30: 3.3V, Mizz_lib:LED_0603, symbol device:LED
- added Q1, Q2, Q3, Q6: MOSFET_P, symbol device:MOSFET_P
- added Q7: MOSFET_N, symbol device:MOSFET_N
- added R69, R71: 10k, Resistors_SMD:R_0603, symbol device:R
- added R70: 10, Resistors_SMD:R_0603, symbol device:R
- D18: value 12V -> BUS_5V; footprint LEDs:LED_0603 -> Mizz_lib:LED_0603
- D19: footprint LEDs:LED_0603 -> Mizz_lib:LED_0603
- P10: value 5V -> XA2_12V; footprint RP_KiCAD_Connector:XA_2T -> Mizz_lib:XA_2T
- P17: value 12V -> XA2_5V; footprint RP_KiCAD_Connector:XA_2T -> Mizz_lib:XA_2T
- Q4, Q5: footprint Mizz_lib:SOT-123 -> (none)
- R26, R28, R30: value 510 -> 10k
- R27, R29: value 510 -> 10
- R31: value 330 -> 10
- R32: value 10k -> 10
- R33: value 10k -> 1.2k
- R34: value 10 -> 510
- R37: value 10k -> 510
- R44: value 1.2k -> 510
- R65: value 10k -> 330
- SW1: value POWER_ON -> Main_POWER
Connections:
- net labels added: XA2_12V, XA2_5V, XA_12V
- net labels removed: CAN0_BUS_12V, CAN1_BUS_12V, CAN_BUS_5V, XA4-12V
- wire segments 406 -> 399
Other:
- moved on the sheet: C18, C19, C42, C5, C6, C7, D14, D15, D26, D29, D32, D35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

Commit message: main 完成
Parts:
- removed Q7: MOSFET_N, symbol device:MOSFET_N
- added D27, D28: DIODE, Mizz_lib:SOD-123, symbol device:DIODE
- added D31: 3.3V, Mizz_lib:LED_0603, symbol device:LED
- added JP4: SWD_3.3V_JP, Mizz_lib:GS2, symbol device:JUMPER
- added Q7: FET_N, Mizz_lib:SOT-23, symbol Hori_lib:MOSFET_N_123
- added R72: 330, Mizz_lib:R_0603, symbol device:R
- C1, C10, C11, C12, C13, C14, C15, C16, C17, C18, C19, C2, C20, C21, C22, C23, C24, C25, C26, C27, C28, C29, C3, C30, C33, C34, C35, C36, C37, C38, C39, C4, C40, C41, C42, C5, C6, C7, C8, C9: footprint Capacitors_SMD:C_0603 -> Mizz_lib:C_0603
- D1: value DATE -> DATA; footprint LEDs:LED_0603 -> Mizz_lib:LED_0603
- D2, D21, D22, D23, D24, D25, D3, D35, D4, D5: footprint LEDs:LED_0603 -> Mizz_lib:LED_0603
- D30: value 3.3V -> 5V
- IC1: footprint Housings_QFP:LQFP-44_10x10mm_Pitch0.8mm -> Mizz_lib:LQFP-44_10x10mm_Pitch0.8mm
- JP1, JP2: footprint Pin_Headers:Pin_Header_Straight_1x02 -> Mizz_lib:Pin_Header_Straight_1x02
- JP3: footprint Connect:GS2 -> Mizz_lib:GS2
- L1: footprint Inductors:Inductor_Taiyo-Yuden_NR-50xx_HandSoldering -> Mizz_lib:Inductor_Taiyo-Yuden_NR-50xx_HandSoldering
- P1: footprint RP_KiCAD_Connector:ZH_6T -> Mizz_lib:ZH_6T
- P11, P12, P15, P16, P4, P6, P8, P9: footprint RP_KiCAD_Connector:XA_4T -> Mizz_lib:XA_4T
- P13, P14, P27: footprint RP_KiCAD_Connector:XA_4LC -> Mizz_lib:XA_4LC
- P18: footprint Pin_Headers:Pin_Header_Straight_1x05 -> Mizz_lib:Pin_Header_Straight_1x05
- P23, P24: footprint Pin_Headers:Pin_Header_Straight_1x10 -> Mizz_lib:Pin_Header_Straight_1x10
- P25, P26: footprint Pin_Headers:Pin_Header_Straight_2x10 -> Mizz_lib:Pin_Header_Straight_2x10
- P28, P29: footprint Pin_Headers:Pin_Header_Straight_1x04 -> Mizz_lib:Pin_Header_Straight_1x04
- P3: value ENC1 -> ENC0; footprint RP_KiCAD_Connector:XA_4T -> Mizz_lib:XA_4T
- P30, P31: footprint Pin_Headers:Pin_Header_Straight_2x04 -> Mizz_lib:Pin_Header_Straight_2x04
- P7: value ENC0 -> ENC1; footprint RP_KiCAD_Connector:XA_4T -> Mizz_lib:XA_4T
- Q1, Q2, Q3, Q6: value MOSFET_P -> FET_P; footprint (none) -> Mizz_lib:SOT-23
- Q4, Q5: footprint (none) -> Mizz_lib:SOT-123
- R1, R10, R11, R12, R13, R14, R15, R16, R17, R18, R19, R20, R21, R22, R23, R24, R25, R26, R27, R28, R29, R30, R31, R32, R33, R34, R35, R36, R37, R38, R39, R4, R40, R41, R42, R43, R44, R45, R46, R47, R48, R49, R5, R50, R51, R52, R53, R54, R55, R56, R57, R58, R59, R6, R60, R61, R62, R63, R64, R66, R67, R68, R69, R7, R70, R71, R8, R9: footprint Resistors_SMD:R_0603 -> Mizz_lib:R_0603
- R2, R3: value 510 -> 330; footprint Resistors_SMD:R_0603 -> Mizz_lib:R_0603
- R65: value 330 -> 510; footprint Resistors_SMD:R_0603 -> Mizz_lib:R_0603
- SW2, SW3, SW4, SW5: footprint Buttons_Switches_SMD:SW_SPST_EVPBF -> Mizz_lib:SW_SPST_PTS645
- U1: footprint Housings_QFP:LQFP-100_14x14mm_Pitch0.5mm -> Mizz_lib:TQFP-100_14x14mm_Pitch0.5mm
- U12: footprint Housings_DIP:DIP-8_W7.62mm -> Mizz_lib:DIP-8_W7.62mm
- U2: footprint Mylib_Device:AZ1086H -> Mizz_lib:AZ1086H
- U3: footprint Housings_SOIC:SOIC-14_3.9x8.7mm_Pitch1.27mm -> Mizz_lib:SOIC-14_3.9x8.7mm_Pitch1.27mm
- U5, U6: footprint Housings_SOIC:SOIC-8_3.9x4.9mm_Pitch1.27mm -> Mizz_lib:SOIC-8_3.9x4.9mm_Pitch1.27mm
- X1: footprint Crystals:Crystal_SMD_5032_2Pads -> Mizz_lib:Crystal_SMD_5032_2Pads
Connections:
- net labels removed: +5C, 5V, XA_5V
- wire segments 399 -> 415
Other:
- moved on the sheet: C11, C12, C13, C18, C19, C26, C27, C33, C34, C35, C36, C37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

Commit message: 完成,製造ファイル生成
Parts:
- removed U11: LOGO, Mizz_lib:PPTP_uva_silk_20x18, symbol myDevice:LOGO
- U13: footprint Mizz_lib:Enc_19.3x7.0_silk -> Mizz_lib:Robocon2019_18.8x18.8_silk
Other:
- moved on the sheet: U10, U13, U9
Changed lines of the file:
@@
 NRST
 $Comp
-L myDevice:LOGO U11
-U 1 1 5DCAD440
+L myDevice:LOGO U10
+U 1 1 5DCADB10
 P 22100 1200
-F 0 "U11" H 22378 1253 60  0000 L CNN
+F 0 "U10" H 22378 1253 60  0000 L CNN
 F 1 "LOGO" H 22378 1147 60  0000 L CNN
-F 2 "Mizz_lib:PPTP_uva_silk_20x18" H 22100 1200 60  0001 C CNN
+F 2 "Mizz_lib:kitLogo_Mask_5.0x5.0" H 22100 1200 60  0001 C CNN
 F 3 "" H 22100 1200 60  0000 C CNN
 	1    22100 1200
@@
 $EndComp
 $Comp
-L myDevice:LOGO U10
-U 1 1 5DCADB10
+L myDevice:LOGO U9
+U 1 1 5DCAEEAA
 P 21250 1200
-F 0 "U10" H 21528 1253 60  0000 L CNN
+F 0 "U9" H 21528 1253 60  0000 L CNN
 F 1 "LOGO" H 21528 1147 60  0000 L CNN
-F 2 "Mizz_lib:kitLogo_Mask_5.0x5.0" H 21250 1200 60  0001 C CNN
+F 2 "Mizz_lib:Mini_Monster" H 21250 1200 60  0001 C CNN
 F 3 "" H 21250 1200 60  0000 C CNN
 	1    21250 1200
-	1    0    0    -1
-$EndComp
-$Comp
-L myDevice:LOGO U9
-U 1 1 5DCAEEAA
-P 20400 1200
-F 0 "U9" H 20678 1253 60  0000 L CNN
-F 1 "LOGO" H 20678 1147 60  0000 L CNN
-F 2 "Mizz_lib:Mini_Monster" H 20400 1200 60  0001 C CNN
-F 3 "" H 20400 1200 60  0000 C CNN
-	1    20400 1200
 	1    0    0    -1
 $EndComp
@@
 L myDevice:LOGO U13
 U 1 1 5C5FBB63
-P 19550 1200
-F 0 "U13" H 19828 1253 60  0000 L CNN
-F 1 "LOGO" H 19828 1147 60  0000 L CNN
-F 2 "Mizz_lib:Enc_19.3x7.0_silk" H 19550 1200 60  0001 C CNN
-F 3 "" H 19550 1200 60  0000 C CNN
-	1    19550 1200
-	1    0    0    -1
-$EndComp
+P 20400 1200
+F 0 "U13" H 20678 1253 60  0000 L CNN
+F 1 "LOGO" H 20678 1147 60  0000 L CNN
+F 2 "Mizz_lib:Robocon2019_18.8x18.8_silk" H 20400 1200 60  0001 C CNN
+F 3 "" H 20400 1200 60  0000 C CNN
+	1    20400 1200
+	1    0    0    -1
+$EndComp

Commit message: あ～、ミスを見つけてしまったよ．なえる．
Parts:
- added C31: 10u, Mizz_lib:C_0603, symbol device:C
- C6: value 22u -> 10u
- D10, D11, D12, D14, D15, D20, D26, D27, D28, D29, D32, D38, D39, D40, D6, D7, D8, D9: symbol device:DIODE -> stm32f4_Centaurus-rescue:DIODE-device
- D3: value SERIAL1_RX -> SERIAL1_TX
- D4: value SERIAL1_TX -> SERIAL1_RX
- JP4: value SWD_3.3V_JP -> PICKit_JP
- Q1, Q2, Q3, Q6: symbol device:MOSFET_P -> stm32f4_Centaurus-rescue:MOSFET_P-device
- Q4, Q5: symbol device:NPN -> stm32f4_Centaurus-rescue:NPN-device
- Q7: symbol Hori_lib:MOSFET_N_123 -> stm32f4_Centaurus-rescue:MOSFET_N_123-Hori_lib
- U10, U13, U9: symbol myDevice:LOGO -> stm32f4_Centaurus-rescue:LOGO-myDevice
- U5, U6: symbol myDevice:MAX3051 -> stm32f4_Centaurus-rescue:MAX3051-myDevice
- U7: symbol Miz:AQM1602_BL -> stm32f4_Centaurus-rescue:AQM1602_BL-Miz
- U8: symbol myDevice:OSTBABS4C2B -> stm32f4_Centaurus-rescue:OSTBABS4C2B-myDevice
Connections:
- net +3.3V: now also C31.1
- net GND: now also Q5.2 (E), U2.1 (GND), C31.2; no longer R43.2
- net at U7.11 (Kathode): now also R43.1; no longer Q5.3 (C)
- new net: Q5.3 (C), R43.2
Other:
- moved on the sheet: Q5, R42, R43
Changed lines of the file:
@@
 P 10625 2300
 F 0 "C6" H 10740 2338 40  0000 L CNN
-F 1 "22u" H 10740 2262 40  0000 L CNN
+F 1 "10u" H 10740 2262 40  0000 L CNN
 F 2 "Mizz_lib:C_0603" H 10663 2150 30  0001 C CNN
 F 3 "" H 10625 2300 60  0000 C CNN
@@
 L power:+3.3V #PWR0115
 U 1 1 5C55D6BD
-P 11525 2100
-F 0 "#PWR0115" H 11525 2060 30  0001 C CNN
-F 1 "+3.3V" H 11534 2238 30  0000 C CNN
-F 2 "" H 11525 2100 60  0000 C CNN
-F 3 "" H 11525 2100 60  0000 C CNN
-	1    11525 2100
+P 11850 2100
+F 0 "#PWR0115" H 11850 2060 30  0001 C CNN
+F 1 "+3.3V" H 11859 2238 30  0000 C CNN
+F 2 "" H 11850 2100 60  0000 C CNN
+F 3 "" H 11850 2100 60  0000 C CNN
+	1    11850 2100
 	1    0    0    -1
 $EndComp
@@
 $EndComp
 $Comp
-L power:GND #PWR0116
-U 1 1 5C55DE40
-P 11075 2525
-F 0 "#PWR0116" H 11075 2525 30  0001 C CNN
-F 1 "GND" H 11075 2455 30  0001 C CNN
-F 2 "" H 11075 2525 60  0000 C CNN
-F 3 "" H 11075 2525 60  0000 C CNN
-	1    11075 2525
-	1    0    0    -1
-$EndComp
-$Comp
 L device:C C5
 U 1 1 5C55E033
@@
 	1    0    0    -1
 $EndComp
-Wire Wire Line
-	11525 2500 11075 2500
-Connection ~ 11075 2500
-Wire Wire Line
-	11075 2500 10625 2500
-Wire Wire Line
-	11075 2500 11075 2525
 $Comp
-L myDevice:MAX3051 U5
+L stm32f4_Centaurus-rescue:MAX3051-myDevice U5
 U 1 1 5C55F62D
 P 18200 7825
@@
 $EndComp
 $Comp
-L myDevice:MAX3051 U6
+L stm32f4_Centaurus-rescue:MAX3051-myDevice U6
 U 1 1 5C55F6F9
 P 18200 8775
@@
 P 3625 13350
 F 0 "D3" H 3625 13175 50  0000 C CNN
-F 1 "SERIAL1_RX" H 3625 13250 50  0000 C CNN
+F 1 "SERIAL1_TX" H 3625 13250 50  0000 C CNN
 F 2 "Mizz_lib:LED_0603" H 3625 13350 60  0001 C CNN
 F 3 "" H 3625 13350 60  0000 C CNN
@@
 P 3625 13625
 F 0 "D4" H 3625 13450 50  0000 C CNN
-F 1 "SERIAL1_TX" H 3625 13525 50  0000 C CNN
+F 1 "SERIAL1_RX" H 3625 13525 50  0000 C CNN
 F 2 "Mizz_lib:LED_0603" H 3625 13625 60  0001 C CNN
 F 3 "" H 3625 13625 60  0000 C CNN
@@
 Connection ~ 5950 3650
 $Comp
-L device:DIODE D14
+L stm32f4_Centaurus-rescue:DIODE-device D14
 U 1 1 5C69879B
 P 5600 2925
@@
 $EndComp
 $Comp
-L device:DIODE D15
+L stm32f4_Centaurus-rescue:DIODE-device D15
 U 1 1 5C6CB8CA
 P 6175 3325
@@
 Connection ~ 4175 15075
 $Comp
-L Miz:AQM1602_BL U7
+L stm32f4_Centaurus-rescue:AQM1602_BL-Miz U7
 U 1 1 5C850363
 P 21700 5100
@@
 L device:R R43
 U 1 1 5C850E36
-P 21250 6250
-F 0 "R43" H 21328 6288 40  0000 L CNN
-F 1 "120" H 21328 6212 40  0000 L CNN
-F 2 "Mizz_lib:R_0603" V 21180 6250 30  0001 C CNN
-F 3 "" H 21250 6250 30  0000 C CNN
-	1    21250 6250
+P 21250 5850
+F 0 "R43" H 21328 5888 40  0000 L CNN
+F 1 "120" H 21328 5812 40  0000 L CNN
+F 2 "Mizz_lib:R_0603" V 21180 5850 30  0001 C CNN
+F 3 "" H 21250 5850 30  0000 C CNN
+	1    21250 5850
 	1    0    0    -1
 $EndComp
@@
 L device:R R42
 U 1 1 5C8510F6
-P 20800 5900
-F 0 "R42" V 20608 5900 40  0000 C CNN
-F 1 "10" V 20684 5900 40  0000 C CNN
-F 2 "Mizz_lib:R_0603" V 20730 5900 30  0001 C CNN
-F 3 "" H 20800 5900 30  0000 C CNN
-	1    20800 5900
+P 20800 6200
+F 0 "R42" V 20608 6200 40  0000 C CNN
+F 1 "10" V 20684 6200 40  0000 C CNN
+F 2 "Mizz_lib:R_0603" V 20730 6200 30  0001 C CNN
+F 3 "" H 20800 6200 30  0000 C CNN
+	1    20800 6200
 	0    1    1    0
 $EndComp
@@
 	18200 5600 18200 5625
 $Comp
-L myDevice:OSTBABS4C2B U8
+L stm32f4_Centaurus-rescue:OSTBABS4C2B-myDevice U8
 U 1 1 5C9A05DA
 P 18725 4775
@@
 $EndComp
 $Comp
-L device:DIODE D20
+L stm32f4_Centaurus-rescue:DIODE-device D20
 U 1 1 5D0368B7
 P 21125 3300
@@
 NRST
 $Comp
-L myDevice:LOGO U10
+L stm32f4_Centaurus-rescue:LOGO-myDevice U10
 U 1 1 5DCADB10
 P 22100 1200
@@
 $EndComp
 $Comp
-L myDevice:LOGO U9
+L stm32f4_Centaurus-rescue:LOGO-myDevice U9
 U 1 1 5DCAEEAA
 P 21250 1200
@@
 Wire Wire Line
 	20800 5000 20800 4700
-Text Label 20650 5900 2    50   ~ 0
+Text Label 20650 6200 2    50   ~ 0
 PB2
 Text Label 3400 8725 2    50   ~ 0
@@
 $EndComp
 $Comp
-L device:DIODE D26
+L stm32f4_Centaurus-rescue:DIODE-device D26
 U 1 1 5E6CB6C3
 P 16400 3650
@@
 Connection ~ 3850 13350
 $Comp
-L myDevice:LOGO U13
+L stm32f4_Centaurus-rescue:LOGO-myDevice U13
 U 1 1 5C5FBB63
 P 20400 1200
@@
 $EndComp
 $Comp
-L device:DIODE D29
+L stm32f4_Centaurus-rescue:DIODE-device D29
 U 1 1 5C73222C
 P 5625 3525
@@
 CAN0_BUS_Vdd
 $Comp
-L device:DIODE D38
+L stm32f4_Centaurus-rescue:DIODE-device D38
 U 1 1 5C7DBE40
 P 21875 8175
@@
 CAN1_BUS_Vdd
 $Comp
-L device:DIODE D39
+L stm32f4_Centaurus-rescue:DIODE-device D39
 U 1 1 5C8C2D01
 P 21875 9125
@@
 $EndComp
 $Comp
-L device:DIODE D32
+L stm32f4_Centaurus-rescue:DIODE-device D32
 U 1 1 5CA9F856
 P 15675 4450
@@
 	2375 5800 2400 5800
 $Comp
-L device:DIODE D40
+L stm32f4_Centaurus-rescue:DIODE-device D40
 U 1 1 5C8AE758
 P 2200 5900
@@
 $EndComp
 $Comp
-L device:NPN Q4
+L stm32f4_Centaurus-rescue:NPN-device Q4
 U 1 1 5C9E9BA8
 P 20825 3700
@@
 Connection ~ 20925 3500
 $Comp
-L device:NPN Q5
+L stm32f4_Centaurus-rescue:NPN-device Q5
 U 1 1 5C9EA261
-P 21150 5900
-F 0 "Q5" H 21341 5999 50  0000 L CNN
-F 1 "NPN" H 21341 5908 50  0000 L CNN
-F 2 "Mizz_lib:SOT-123" H 21150 5900 60  0001 C CNN
-F 3 "transistors/bipolar/*.*" H 21341 5809 60  0000 L CNN
-	1    21150 5900
+P 21150 6200
+F 0 "Q5" H 21341 6299 50  0000 L CNN
+F 1 "NPN" H 21341 6208 50  0000 L CNN
+F 2 "Mizz_lib:SOT-123" H 21150 6200 60  0001 C CNN
+F 3 "transistors/bipolar/*.*" H 21341 6109 60  0000 L CNN
+	1    21150 6200
 	1    0    0    -1
 $EndComp
@@
 $EndComp
 $Comp
-L device:DIODE D8
+L stm32f4_Centaurus-rescue:DIODE-device D8
 U 1 1 5CB3AB03
 P 2650 2050
@@
 $EndComp
 $Comp
-L device:DIODE D11
+L stm32f4_Centaurus-rescue:DIODE-device D11
 U 1 1 5CB410C0
 P 5800 2500
@@
 $EndComp
 $Comp
-L device:DIODE D6
+L stm32f4_Centaurus-rescue:DIODE-device D6
 U 1 1 5CB4A23E
 P 3125 2050
@@
 $EndComp
 $Comp
-L device:MOSFET_P Q1
+L stm32f4_Centaurus-rescue:MOSFET_P-device Q1
 U 1 1 5CB4B628
 P 3375 2275
@@
 CAN_BUS_12V
 $Comp
-L device:DIODE D7
+L stm32f4_Centaurus-rescue:DIODE-device D7
 U 1 1 5CB4D7AA
 P 3475 2675
@@
 $EndComp
 $Comp
-L device:DIODE D9
+L stm32f4_Centaurus-rescue:DIODE-device D9
 U 1 1 5CCEB104
 P 6300 2500
@@
 $EndComp
 $Comp
-L device:MOSFET_P Q2
+L stm32f4_Centaurus-rescue:MOSFET_P-device Q2
 U 1 1 5CCEC522
 P 6525 2725
@@
 $EndComp
 $Comp
-L device:DIODE D10
+L stm32f4_Centaurus-rescue:DIODE-device D10
 U 1 1 5CCEC6BA
 P 6625 3125
@@
 $EndComp
 $Comp
-L device:MOSFET_P Q3
+L stm32f4_Centaurus-rescue:MOSFET_P-device Q3
 U 1 1 5CDC70D4
 P 7825 2700
@@
 $EndComp
 $Comp
-L device:DIODE D12
+L stm32f4_Centaurus-rescue:DIODE-device D12
 U 1 1 5CE4523A
 P 7925 3100
@@
 $EndComp
 $Comp
-L device:MOSFET_P Q6
+L stm32f4_Centaurus-rescue:MOSFET_P-device Q6
 U 1 1 5CE47413
 P 9425 2300
@@
 Connection ~ 7925 2500
 $Comp
-L device:DIODE D27
+L stm32f4_Centaurus-rescue:DIODE-device D27
 U 1 1 5D033C0D
 P 7600 2500
@@
 Connection ~ 22425 12550
 $Comp
-L device:DIODE D28
+L stm32f4_Centaurus-rescue:DIODE-device D28
 U 1 1 5D3C34DF
 P 20725 10475
@@
 P 21025 10675
 F 0 "JP4" H 21025 10931 60  0000 C CNN
-F 1 "SWD_3.3V_JP" H 21025 10840 40  0000 C CNN
+F 1 "PICKit_JP" H 21025 10840 40  0000 C CNN
 F 2 "Mizz_lib:GS2" H 21025 10675 60  0001 C CNN
 F 3 "" H 21025 10675 60  0000 C CNN
@@
 $EndComp
 $Comp
-L Hori_lib:MOSFET_N_123 Q7
+L stm32f4_Centaurus-rescue:MOSFET_N_123-Hori_lib Q7
 U 1 1 5C8EBE40
 P 16100 3750
@@
 Connection ~ 9525 2100
 Connection ~ 11525 2100
-Wire Wire Line
-	9525 2100 10625 2100
 Connection ~ 10625 2100
 $Comp
@@
 	13350 3550 13350 3900
 Connection ~ 13350 3900
+$Comp
+L device:C C31
+U 1 1 5CC6C1DB
+P 11850 2300
+F 0 "C31" H 11965 2338 40  0000 L CNN
+F 1 "10u" H 11965 2262 40  0000 L CNN
+F 2 "Mizz_lib:C_0603" H 11888 2150 30  0001 C CNN
+F 3 "" H 11850 2300 60  0000 C CNN
+	1    11850 2300
+	1    0    0    -1
+$EndComp
+$Comp
+L power:GND #PWR0116
+U 1 1 5CCA08C1
+P 11075 2575
+F 0 "#PWR0116" H 11075 2575 30  0001 C CNN
+F 1 "GND" H 11075 2505 30  0001 C CNN
+F 2 "" H 11075 2575 50  0001 C CNN
+F 3 "" H 11075 2575 50  0001 C CNN
+	1    11075 2575
+	1    0    0    -1
+$EndComp
+Wire Wire Line
+	11075 2575 11075 2550
+Wire Wire Line
+	11075 2550 11525 2550
+Wire Wire Line
+	11525 2550 11525 2500
+Connection ~ 11075 2550
+Wire Wire Line
+	11075 2550 10625 2550
+Wire Wire Line
+	10625 2500 10625 2550
+Wire Wire Line
+	9525 2100 10625 2100
+Wire Wire Line
+	11525 2100 11850 2100
+Connection ~ 11850 2100
+Wire Wire Line
+	11525 2550 11850 2550
+Wire Wire Line
+	11850 2550 11850 2500
+Connection ~ 11525 2550
 $EndSCHEMATC

Commit message: とりあえず、問題なければ完了.
Parts:
- removed R27, R29, R31, R32, R70: 10, Mizz_lib:R_0603, symbol device:R
- added JP5: I/O_Vdd, Mizz_lib:Pin_Header_Straight_1x03, symbol device:JUMPER3
- P28: value I/O_3.3V -> I/O_5V
- P29: value I/O_5V -> I/O_Variable
- P30: value I/O_3.3V_batt -> I/O_5V_batt
- P31: value I/O_5V_batt -> I/O_Variable
- U13: footprint Mizz_lib:Robocon2019_18.8x18.8_silk -> Mizz_lib:Robocon2019_30.0x30.0_silk
Connections:
- net +3.3V: now also JP5.1; no longer P30.1 (P1), P30.3 (P3), P30.5 (P5), P30.7 (P7)
- net +5V: now also P30.1 (P1), P30.3 (P3), P30.5 (P5), P30.7 (P7), JP5.3; no longer P31.1 (P1), P31.3 (P3), P31.5 (P5), P31.7 (P7)
- net GND: now also Q4.2 (E); no longer R53.2
- net USART2_RX: now also IC1.2 (RP22_CN18_RC6); no longer IC1.3 (RP23_CN17_RC7)
- net USART2_TX: now also IC1.3 (RP23_CN17_RC7); no longer IC1.2 (RP22_CN18_RC6)
- net XA_12V: now also Q1.1 (G)
- net at P27.4 (P4), R71.1: now also Q7.1 (G)
- net at R53.1: now also D20.1 (A), SP1.2; no longer Q4.2 (E)
- net at D11.2 (K), D9.1 (A), R28.1: now also Q2.1 (G)
- net at D27.1 (A), D9.2 (K), Q2.3 (D)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: now also Q3.1 (G)
- net at SW1.2: now also Q6.1 (G)
- new net: JP5.2, P31.1 (P1), P31.3 (P3), P31.5 (P5), P31.7 (P7)
- new net: Q4.3 (C), R53.2
Other:
- moved on the sheet: C31, C6, C7, D7, Q1, Q4, Q6, R51, R53, U2
