File: stm32f4_Centaurus_ver.1.0/stm32f4_Centaurus/stm32f4_Centaurus.kicad_pcb (KiCad board)
At the start: 2 copper layers, 100 x 95 mm, 207 parts, among them IC1 PIC24FJ64GB004, P1 PICKit3, P10 5V, P11 CAN0, P12 CAN1, P13 CAN0, P14 CAN1, P15 SERIAL2, P16 SERIAL0, P17 12V, P18 SWD, P2 SERIAL5_SBDBT, P23 A/D, P24 PWM, P25 A/D_batt, P26 PWM_batt, P27 EMERGENCY_CHECK, P28 I/O_3.3V, P29 I/O_5V, P3 ENC1, P30 I/O_3.3V_batt, P31 I/O_5V_batt, P4 ENC2, P5 SERIAL1, P6 ENC3, P7 ENC0, P8 SERIAL4, P9 SERIAL3, Q1 P_FET, Q2 P_FET, Q3 P_FET, Q4 NPN, Q5 NPN, Q6 P_FET, SW1 POWER_ON, SW2 SW1, SW3 SW0, SW4 SW2, SW5 SW3, U1 STM32F407VG, U10 LOGO, U11 LOGO, U12 25LC010A, U13 LOGO, U2 AZ1086H, U3 MCP2221A, U4 AP3211, U5 MAX3051, U6 MAX3051, U7 AQM1602_BL, U8 OSTBABS4C2B, U9 LOGO, X1 8MHz

Commit message: RC19 mains.
Parts:
- removed D27, D28: DIODE, Mizz_lib:SOD-123
- added R69: 10k, Resistors_SMD:R_0603, F.Cu at (225.5, 28.6)
- added R70: 10, Resistors_SMD:R_0603, F.Cu at (238.1, 20.8)
- added R71: 10k, Resistors_SMD:R_0603, F.Cu at (240.8, 20.8)
- D10: value USE_5V -> DIODE; footprint LEDs:LED_0603 -> Mizz_lib:SOD-123
- D11: value 3.3V -> DIODE; footprint LEDs:LED_0603 -> Mizz_lib:SOD-123
- D13: value DIODE -> XA2_12V; footprint Mizz_lib:SOD-123 -> Mizz_lib:LED_0603; moved to F.Cu
- D16: value DIODE -> XA_5V; footprint Mizz_lib:SOD-123 -> Mizz_lib:LED_0603; moved to F.Cu
- D17: value DIODE -> 12V_to_5V; footprint Mizz_lib:SOD-123 -> Mizz_lib:LED_0603; moved to F.Cu
- D18: value 12V -> BUS_5V; footprint LEDs:LED_0603 -> Mizz_lib:LED_0603
- D19: footprint LEDs:LED_0603 -> Mizz_lib:LED_0603
- D30: value DIODE -> 3.3V; footprint Mizz_lib:SOD-123 -> Mizz_lib:LED_0603
- D6: value SELF_5V -> DIODE; footprint LEDs:LED_0603 -> Mizz_lib:SOD-123
- D7: value BUS_5V -> DIODE; footprint LEDs:LED_0603 -> Mizz_lib:SOD-123
- D8: value 12V_to_5V -> DIODE; footprint LEDs:LED_0603 -> Mizz_lib:SOD-123
- D9: value SW_5V -> DIODE; footprint LEDs:LED_0603 -> Mizz_lib:SOD-123
- P10: value 5V -> XA2_12V; footprint RP_KiCAD_Connector:XA_2T -> Mizz_lib:XA_2T
- P17: value 12V -> XA2_5V; footprint RP_KiCAD_Connector:XA_2T -> Mizz_lib:XA_2T
- Q1, Q2, Q3, Q6: value P_FET -> MOSFET_P
- R26, R28, R30: value 510 -> 10k
- R27, R29: value 510 -> 10
- R31: value 330 -> 10
- R32: value 10k -> 10
- R33: value 10k -> 1.2k
- R34: value 10 -> 510
- R37: value 10k -> 510
- R44: value 1.2k -> 510
- R65: value 10k -> 330
- SW1: value POWER_ON -> Main_POWER
- moved U11 132.2 mm to (213.9, 36.6)
- moved U7 50.2 mm to (24.2, 64.6)
- moved U13 44.2 mm to (22.2, 43.4)
- moved Q6 43.1 mm to (63.2, 128.5), turned to 90 degrees
- moved D17 37.5 mm to (45.8, 110.0), turned to 90 degrees
- moved Q1 32.8 mm to (43.5, 115.0)
- moved U10 31.1 mm to (36.3, 48.3)
- moved D18 27.7 mm to (81.0, 141.5)
- moved R13 23.0 mm to (169.2, 75.2)
- moved R14 23.0 mm to (169.2, 77.0)
- moved R18 23.0 mm to (169.2, 78.9)
- moved R20 23.0 mm to (169.2, 73.5)
- moved D13 22.8 mm to (56.8, 127.2), turned to 0 degrees
- moved D16 22.4 mm to (56.8, 130.1), turned to 0 degrees
- moved P26 18.0 mm to (61.8, 66.8)
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Connections:
- net /USART4_RX renamed /UART4_RX
- net /USART4_TX renamed /UART4_TX
- D10 pad 1: Net-(D10-Pad1) -> /12V_TO_5V
- D10 pad 2: GND -> Net-(D10-Pad2)
- D11 pad 1: Net-(D11-Pad1) -> XA2_5V
- D11 pad 2: GND -> /XA_5V
- D12 pad 1: /XA_5V -> /BUS_5V
- D12 pad 2: /5V -> Net-(D12-Pad2)
- D13 pad 1: /BUS_5V -> Net-(D13-Pad1)
- D13 pad 2: Net-(D13-Pad2) -> GND
- D16 pad 1: /5V -> Net-(D16-Pad1)
- D16 pad 2: +5C -> GND
- D17 pad 1: /CAN_BUS_5V -> Net-(D17-Pad1)
- D17 pad 2: Net-(D17-Pad2) -> GND
- D30 pad 1: /XA4-12V -> Net-(D30-Pad1)
- D30 pad 2: +12V -> GND
- D32 pad 2: /XA4-12V -> /XA_12V
- D38 pad 2: /CAN0_BUS_12V -> /CAN_BUS_12V
- D39 pad 2: /CAN1_BUS_12V -> /CAN_BUS_12V
- D40 pad 2: +3.3V -> Net-(D40-Pad2)
- D6 pad 1: /XA_5V -> /XA_12V
- D6 pad 2: Net-(D6-Pad2) -> +12V
- D7 pad 1: Net-(D7-Pad1) -> /CAN_BUS_12V
- D7 pad 2: GND -> Net-(D7-Pad2)
- D8 pad 1: Net-(D8-Pad1) -> XA2_12V
- D8 pad 2: GND -> /XA_12V
- D9 pad 1: Net-(D9-Pad1) -> /XA_5V
- D9 pad 2: GND -> /5V
- JP3 pad 1: Net-(D40-Pad1) -> +3.3V
- JP3 pad 2: Net-(JP3-Pad2) -> Net-(D40-Pad2)
- P10 pad 2: /XA_5V -> XA2_12V
- P17 pad 2: +12V -> XA2_5V
- P18 pad 2: Net-(JP3-Pad2) -> Net-(D40-Pad1)
- P27 pad 4: /PB11 -> Net-(P27-Pad4)
- Q1 pad 1: /XA_5V -> Net-(Q1-Pad1)
- Q1 pad 2: Net-(D13-Pad2) -> Net-(D7-Pad2)
- Q1 pad 3: /5V -> +12V
- Q2 pad 2: +5C -> Net-(D10-Pad2)
- Q2 pad 3: +5V -> /5V
- Q3 pad 1: /5V -> Net-(Q3-Pad1)
- Q3 pad 2: Net-(D17-Pad2) -> Net-(D12-Pad2)
- Q4 pad 3: Net-(Q4-Pad3) -> Net-(D20-Pad1)
- Q5 pad 3: Net-(D20-Pad1) -> Net-(Q5-Pad3)
- Q6 pad 1: /XA4-12V -> Net-(Q6-Pad1)
- Q6 pad 2: Net-(D31-Pad2) -> +5C
- Q6 pad 3: +12V -> +5V
- R26 pad 1: GND -> /XA_12V
- R26 pad 2: Net-(D6-Pad2) -> GND
- R27 pad 1: Net-(D7-Pad1) -> Net-(Q1-Pad1)
- R27 pad 2: /BUS_5V -> /XA_12V
- R28 pad 1: Net-(D8-Pad1) -> /XA_5V
- R28 pad 2: /12V_TO_5V -> Net-(R28-Pad2)
- R29 pad 1: Net-(D9-Pad1) -> Net-(Q2-Pad1)
- R29 pad 2: +5C -> /XA_5V
- R30 pad 1: Net-(D10-Pad1) -> /5V
- R30 pad 2: +5V -> GND
- R31 pad 1: Net-(D11-Pad1) -> Net-(Q3-Pad1)
- R31 pad 2: +3.3V -> /5V
- R32 pad 1: Net-(R32-Pad1) -> Net-(Q6-Pad1)
- R32 pad 2: GND -> Net-(R32-Pad2)
- R33 pad 1: /XA_5V -> Net-(D13-Pad1)
- R33 pad 2: GND -> XA2_12V
- R34 pad 1: Net-(Q2-Pad1) -> Net-(D16-Pad1)
- R34 pad 2: Net-(R34-Pad2) -> XA2_5V
- R37 pad 1: /5V -> Net-(D17-Pad1)
- R37 pad 2: GND -> /12V_TO_5V
- R42 pad 1: Net-(Q4-Pad1) -> Net-(Q5-Pad1)
- R43 pad 1: Net-(Q4-Pad2) -> Net-(Q5-Pad2)
- R44 pad 2: +12V -> /BUS_5V
- R51 pad 1: Net-(Q5-Pad1) -> Net-(Q4-Pad1)
- R53 pad 1: Net-(Q5-Pad2) -> Net-(Q4-Pad2)
- R65 pad 1: /XA4-12V -> Net-(D30-Pad1)
- R65 pad 2: GND -> +3.3V
- R66 pad 2: /XA4-12V -> XA4_12V
- R67 pad 2: /CAN0_BUS_12V -> CAN0_BUS_Vdd
- R68 pad 2: /CAN1_BUS_12V -> CAN1_BUS_Vdd
- SW1 pad 2: Net-(R34-Pad2) -> Net-(R32-Pad2)
- SW1 pad 3: Net-(R32-Pad1) -> GND
- U7 pad 11: Net-(Q4-Pad3) -> Net-(Q5-Pad3)
Routing:
- net +3.3V: track 466.6 -> 256.8 mm, vias 31 -> 14
- net +5V: track 373.9 -> 255.2 mm, vias 15 -> 5
- net +12V: track 60.9 -> 0.00 mm, vias 2 -> 0
- net /NRST: track 102.1 -> 156.1 mm, vias 7 -> 11
- net /TIM1_CH4: track 75.3 -> 35.0 mm
- net +5C: track 38.8 -> 0.00 mm, vias 1 -> 0
- net /TIM1_CH3: track 72.6 -> 35.3 mm
- net /BUS_5V: track 34.5 -> 0.00 mm, vias 4 -> 0
- net /TIM1_CH2: track 69.6 -> 35.1 mm
- net /TIM1_CH1: track 65.5 -> 35.1 mm
- net /USART1_TX: track 78.4 -> 52.0 mm, vias 2 -> 0
- net /USART1_RX: track 80.1 -> 54.4 mm, vias 2 -> 0
- net /XA_5V: track 23.9 -> 0.00 mm, vias 1 -> 0
- net /UART5_TX: track 70.4 -> 49.2 mm
- net /UART5_RX: track 71.4 -> 50.7 mm, vias 7 -> 6
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Other:
- board text added: "Desgined by A.Mizuta in 2019/02/08."
- board text removed: "*"
- board text removed: "Desgined by A.Mizuta in 2019/02/08. Special Thanks : Y.Shoda, T.Yamada."

Commit message: main 完成
Parts:
- removed D33, D34: DIODE, Mizz_lib:SOD-123
- removed U9: LOGO, Mizz_lib:Mini_Monster
- added D27: DIODE, Mizz_lib:SOD-123, B.Cu at (66.0, 127.8)
- added D28: DIODE, Mizz_lib:SOD-123, B.Cu at (139.9, 118.7)
- added JP4: SWD_3.3V_JP, Mizz_lib:GS2, B.Cu at (140.0, 122.2)
- added Q7: FET_N, Mizz_lib:SOT-23, B.Cu at (67.2, 119.8)
- added R72: 330, Mizz_lib:R_0603, F.Cu at (79.8, 119.5)
- added REF**: Beer_Hall, Mizz_lib:Beer_Hall, F.Cu at (56.0, 62.0)
- added REF**: Beer_Hall, Mizz_lib:Beer_Hall, F.Cu at (56.0, 135.0)
- added REF**: Beer_Hall, Mizz_lib:Beer_Hall, F.Cu at (150.0, 135.0)
- added REF**: Beer_Hall, Mizz_lib:Beer_Hall, F.Cu at (150.0, 62.0)
- C1, C10, C11, C12, C13, C14, C15, C16, C17, C18, C19, C2, C20, C21, C22, C23, C24, C25, C26, C27, C28, C29, C3, C30, C33, C34, C35, C36, C37, C38, C39, C4, C40, C41, C42, C5, C6, C7, C8, C9: footprint Capacitors_SMD:C_0603 -> Mizz_lib:C_0603
- D1: value DATE -> DATA; footprint LEDs:LED_0603 -> Mizz_lib:LED_0603
- D10, D11, D6, D7, D8, D9: moved to B.Cu
- D2, D21, D22, D23, D24, D25, D3, D35, D4, D5: footprint LEDs:LED_0603 -> Mizz_lib:LED_0603
- D30: value 3.3V -> 5V; moved to F.Cu
- D31: value DIODE -> 3.3V; footprint Mizz_lib:SOD-123 -> Mizz_lib:LED_0603; moved to F.Cu
- IC1: footprint Housings_QFP:LQFP-44_10x10mm_Pitch0.8mm -> Mizz_lib:LQFP-44_10x10mm_Pitch0.8mm
- JP1, JP2: footprint Pin_Headers:Pin_Header_Straight_1x02 -> Mizz_lib:Pin_Header_Straight_1x02
- JP3: footprint Connect:GS2 -> Mizz_lib:GS2
- L1: footprint Inductors:Inductor_Taiyo-Yuden_NR-50xx_HandSoldering -> Mizz_lib:Inductor_Taiyo-Yuden_NR-50xx_HandSoldering
- P1: footprint RP_KiCAD_Connector:ZH_6T -> Mizz_lib:ZH_6T
- P11, P12, P15, P16, P4, P6, P8, P9: footprint RP_KiCAD_Connector:XA_4T -> Mizz_lib:XA_4T
- P13, P14, P27: footprint RP_KiCAD_Connector:XA_4LC -> Mizz_lib:XA_4LC
- P18: footprint Pin_Headers:Pin_Header_Straight_1x05 -> Mizz_lib:Pin_Header_Straight_1x05
- P23, P24: footprint Pin_Headers:Pin_Header_Straight_1x10 -> Mizz_lib:Pin_Header_Straight_1x10
- P25, P26: footprint Pin_Headers:Pin_Header_Straight_2x10 -> Mizz_lib:Pin_Header_Straight_2x10
- P28, P29: footprint Pin_Headers:Pin_Header_Straight_1x04 -> Mizz_lib:Pin_Header_Straight_1x04
- P3: value ENC1 -> ENC0; footprint RP_KiCAD_Connector:XA_4T -> Mizz_lib:XA_4T
- P30, P31: footprint Pin_Headers:Pin_Header_Straight_2x04 -> Mizz_lib:Pin_Header_Straight_2x04
- P7: value ENC0 -> ENC1; footprint RP_KiCAD_Connector:XA_4T -> Mizz_lib:XA_4T
- Q1, Q2, Q3, Q6: value MOSFET_P -> FET_P; footprint TO_SOT_Packages_SMD:SOT-23 -> Mizz_lib:SOT-23
- R1, R10, R11, R12, R13, R14, R15, R16, R17, R18, R19, R20, R21, R22, R23, R24, R25, R32, R33, R34, R35, R36, R38, R39, R4, R40, R41, R42, R43, R44, R45, R46, R47, R48, R49, R5, R50, R51, R52, R53, R54, R55, R56, R57, R58, R59, R6, R60, R61, R62, R63, R64, R66, R67, R68, R7, R8, R9: footprint Resistors_SMD:R_0603 -> Mizz_lib:R_0603
- R2, R3: value 510 -> 330; footprint Resistors_SMD:R_0603 -> Mizz_lib:R_0603
- R26, R27, R28, R29, R30, R31, R69, R70, R71: footprint Resistors_SMD:R_0603 -> Mizz_lib:R_0603; moved to B.Cu
- R37: footprint Resistors_SMD:R_0603 -> Mizz_lib:R_0603; moved to F.Cu
- R65: value 330 -> 510; footprint Resistors_SMD:R_0603 -> Mizz_lib:R_0603; moved to F.Cu
- SW2, SW3, SW4, SW5: footprint Buttons_Switches_SMD:SW_SPST_EVPBF -> Mizz_lib:SW_SPST_PTS645
- U1: footprint Housings_QFP:LQFP-100_14x14mm_Pitch0.5mm -> Mizz_lib:TQFP-100_14x14mm_Pitch0.5mm
- U12: footprint Housings_DIP:DIP-8_W7.62mm -> Mizz_lib:DIP-8_W7.62mm
- U2: footprint Mylib_Device:AZ1086H -> Mizz_lib:AZ1086H
- U3: footprint Housings_SOIC:SOIC-14_3.9x8.7mm_Pitch1.27mm -> Mizz_lib:SOIC-14_3.9x8.7mm_Pitch1.27mm
- U5, U6: footprint Housings_SOIC:SOIC-8_3.9x4.9mm_Pitch1.27mm -> Mizz_lib:SOIC-8_3.9x4.9mm_Pitch1.27mm
- X1: footprint Crystals:Crystal_SMD_5032_2Pads -> Mizz_lib:Crystal_SMD_5032_2Pads
- moved R71 201.3 mm to (64.5, 118.0), turned to 270 degrees
- moved R70 196.3 mm to (67.0, 117.0)
- moved R69 177.7 mm to (72.2, 118.5), turned to 180 degrees
- moved U11 117.9 mm to (104.8, 81.0)
- moved U7 73.5 mm to (95.2, 83.5)
- moved U10 42.6 mm to (70.7, 73.4)
- moved D32 35.5 mm to (56.5, 117.0), turned to 180 degrees
- moved C41 33.5 mm to (95.8, 101.8), turned to 90 degrees
- moved U12 33.4 mm to (90.0, 101.5)
- moved R44 32.4 mm to (79.8, 116.5)
- moved D31 32.3 mm to (77.2, 119.5), turned to 0 degrees
- moved P27 31.8 mm to (62.0, 109.8)
- moved D17 31.7 mm to (77.2, 113.5), turned to 0 degrees
- moved R66 31.4 mm to (65.0, 112.0), turned to 180 degrees
- moved D35 30.1 mm to (65.8, 111.0), turned to 270 degrees
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Connections:
- net +5C renamed Net-(D27-Pad2)
- net /5V renamed Net-(D27-Pad1)
- net /XA_5V renamed Net-(D11-Pad2)
- D1 pad 1: +5V -> Net-(D1-Pad1)
- D2 pad 1: +5V -> Net-(D2-Pad1)
- D31 pad 1: /CAN_BUS_12V -> Net-(D31-Pad1)
- D31 pad 2: Net-(D31-Pad2) -> GND
- IC1 pad 14: Net-(IC1-Pad14) -> Net-(D1-Pad2)
- IC1 pad 15: Net-(IC1-Pad15) -> Net-(D2-Pad2)
- P1 pad 2: +5V -> Net-(D28-Pad1)
- R2 pad 1: Net-(D1-Pad2) -> +3.3V
- R2 pad 2: Net-(IC1-Pad14) -> Net-(D1-Pad1)
- R28 pad 2: Net-(R28-Pad2) -> GND
- R3 pad 1: Net-(D2-Pad2) -> +3.3V
- R3 pad 2: Net-(IC1-Pad15) -> Net-(D2-Pad1)
- R42 pad 2: /PE10 -> /PB2
- R65 pad 2: +3.3V -> +5V
- U12 pad 3: /PE7 -> /PE10
- U12 pad 7: /PB2 -> /PE7
- U2 pad 1: GND -> Net-(U2-Pad1)
Routing:
- net +3.3V: track 256.8 -> 431.1 mm, vias 14 -> 31
- net +5V: track 255.2 -> 329.5 mm, vias 5 -> 14
- net /NRST: track 156.1 -> 85.7 mm, vias 11 -> 9
- net Net-(R64-Pad2): track 2.50 -> 48.5 mm, vias 0 -> 7
- net /TIM1_CH4: track 35.0 -> 74.3 mm
- net Net-(R62-Pad1): track 14.8 -> 52.5 mm, vias 2 -> 8
- net /TIM1_CH3: track 35.3 -> 71.8 mm
- net /TIM2_CH1: track 6.95 -> 40.6 mm, vias 1 -> 3
- net /TIM1_CH2: track 35.1 -> 68.6 mm
- net /USART1_TX: track 52.0 -> 84.3 mm, vias 0 -> 3
- net /USART1_RX: track 54.4 -> 86.4 mm, vias 0 -> 3
- net /TIM1_CH1: track 35.1 -> 62.2 mm
- net /TIM12_CH1: track 22.2 -> 48.1 mm
- net +12V: track 0.00 -> 25.9 mm, vias 0 -> 2
- net /TIM2_CH2: track 19.6 -> 45.0 mm
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Other:
- board size 100 x 95 mm -> 100 x 79 mm
- board text added: "*"
- board text added: "1(1602,I2C)"
- board text added: "1(SPI)"
- board text added: "100 x 95(mm x mm)"
- board text added: "4(A-B)"
- board text added: "5V/12V/CAN BUS Vdd"
- board text added: "6(microB,Advanced SBDBT)"
- board text added: "7(RGB,RESET)"
- board text added: "8(3.3V_I/Ox4, 5V_I/O4)"
- board text added: "MCLR"
- board text added: "NC"
- board text added: "PGEC"
- board text added: "PGED"
- board text added: "POWER IN"
- board text added: "Vdd"
- board text added: "________________________________________________________________"
- board text removed: "1(1602)"
- board text removed: "1(SPI BUS)"
- board text removed: "100x95"
- board text removed: "4(AB)"
- board text removed: "5V/12V"
- board text removed: "6(MiniB * 1,SBDBT * 1)"
- board text removed: "7(RGB * 1)"
- board text removed: "8(3.3V * 4, 5V * 4)"
- board text removed: "POWER"
- board text removed: "______________________________________________________________"

Commit message: 完成,製造ファイル生成
Parts:
- removed REF** (x4): Beer_Hall, Mizz_lib:Beer_Hall
- removed U11: LOGO, Mizz_lib:PPTP_uva_silk_20x18
- added U9: LOGO, Mizz_lib:Mini_Monster, F.Cu at (128.0, 89.2)
- U13: footprint Mizz_lib:Enc_19.3x7.0_silk -> Mizz_lib:Robocon2019_18.8x18.8_silk
- moved U13 71.1 mm to (85.0, 76.8)
- moved P1 0.25 mm to (141.8, 114.5)
- moved D19 0.12 mm to (102.0, 114.8)
Routing:
- net /XA_12V: track 5.89 -> 12.5 mm, vias 1 -> 2
- net +3.3V: vias 31 -> 33
- net Net-(D25-Pad2): vias 0 -> 1
- net Net-(D24-Pad2): vias 0 -> 1
- net Net-(D23-Pad2): vias 0 -> 1
- net Net-(D22-Pad2): vias 0 -> 1
- net Net-(D21-Pad2): vias 0 -> 1
- net Net-(D2-Pad1): vias 0 -> 1
- net Net-(D19-Pad2): vias 0 -> 1
- net Net-(D13-Pad1): vias 0 -> 1
- net Net-(D1-Pad1): vias 0 -> 1
- net GND: vias 269 -> 857
- net /TIM5_CH2: vias 3 -> 1
- net /TIM5_CH1: vias 3 -> 2
- net /NRST: vias 9 -> 7
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
Commit message: あ～、ミスを見つけてしまったよ．なえる．
Parts:
- added C31: 10u, Mizz_lib:C_0603, B.Cu at (90.5, 122.0)
- C6: value 22u -> 10u
- D3: value SERIAL1_RX -> SERIAL1_TX
- D4: value SERIAL1_TX -> SERIAL1_RX
- JP4: value SWD_3.3V_JP -> PICKit_JP
Connections:
- Q5 pad 2: Net-(Q5-Pad2) -> GND
- R43 pad 1: Net-(Q5-Pad2) -> Net-(R43-Pad1)
- R43 pad 2: GND -> Net-(Q5-Pad3)
- U2 pad 1: Net-(U2-Pad1) -> GND
- U7 pad 11: Net-(Q5-Pad3) -> Net-(R43-Pad1)
Routing:
- net /SWDIO: track 36.8 -> 30.6 mm
- net Net-(D16-Pad1): vias 1 -> 2
- net GND: vias 857 -> 1212
- net (no net): vias 4 -> 5
Other:
- board text added: "100 x 80(mm x mm)"
- board text added: "2(2.0A)"
- board text added: "ENCODER"
- board text added: "_________________________________________________________________"
- board text removed: "100 x 95(mm x mm)"
- board text removed: "2(2.0B)"
- board text removed: "ENC"
- board text removed: "________________________________________________________________"

Commit message: とりあえず、問題なければ完了.
Parts:
- removed R27, R29, R31, R32, R70: 10, Mizz_lib:R_0603
- added JP5: I/O_Vdd, Mizz_lib:Pin_Header_Straight_1x03, F.Cu at (144.2, 66.8)
- P28: value I/O_3.3V -> I/O_5V
- P29: value I/O_5V -> I/O_Variable
- P30: value I/O_3.3V_batt -> I/O_5V_batt
- P31: value I/O_5V_batt -> I/O_Variable
- U13: footprint Mizz_lib:Robocon2019_18.8x18.8_silk -> Mizz_lib:Robocon2019_30.0x30.0_silk
- moved R53 6.15 mm to (81.0, 106.2)
- moved U13 5.15 mm to (89.8, 78.8)
- moved R43 4.56 mm to (109.8, 90.5), turned to 90 degrees
- moved JP3 3.58 mm to (140.0, 75.0)
- moved D40 3.26 mm to (144.0, 75.0)
- moved Q4 2.36 mm to (83.5, 103.2)
- moved P29 1.75 mm to (132.5, 66.8)
- moved P31 1.75 mm to (132.5, 64.2)
- moved R71 1.06 mm to (65.2, 117.2), turned to 0 degrees
- moved U10 0.96 mm to (69.8, 73.2)
- moved R51 0.90 mm to (85.2, 106.2)
- moved Q5 0.75 mm to (109.8, 87.2)
- moved C11 0.25 mm to (125.2, 73.0)
- moved C13 0.25 mm to (127.8, 73.0)
Connections:
- IC1 pad 2: /USART2_TX -> /USART2_RX
- IC1 pad 3: /USART2_RX -> /USART2_TX
- P30 pad 1: +3.3V -> +5V
- P30 pad 3: +3.3V -> +5V
- P30 pad 5: +3.3V -> +5V
- P30 pad 7: +3.3V -> +5V
- P31 pad 1: +5V -> Net-(JP5-Pad2)
- P31 pad 3: +5V -> Net-(JP5-Pad2)
- P31 pad 5: +5V -> Net-(JP5-Pad2)
- P31 pad 7: +5V -> Net-(JP5-Pad2)
- Q1 pad 1: Net-(Q1-Pad1) -> /XA_12V
- Q2 pad 1: Net-(Q2-Pad1) -> Net-(D11-Pad2)
- Q3 pad 1: Net-(Q3-Pad1) -> Net-(D27-Pad1)
- Q4 pad 2: Net-(Q4-Pad2) -> GND
- Q4 pad 3: Net-(D20-Pad1) -> Net-(Q4-Pad3)
- Q7 pad 1: Net-(Q7-Pad1) -> Net-(P27-Pad4)
- R53 pad 1: Net-(Q4-Pad2) -> Net-(D20-Pad1)
- R53 pad 2: GND -> Net-(Q4-Pad3)
- SW1 pad 2: Net-(R32-Pad2) -> Net-(Q6-Pad1)
Routing:
- net +3.3V: track 431.1 -> 447.5 mm
- net +5V: track 329.5 -> 344.9 mm
- net Net-(JP5-Pad2): track 0.00 -> 11.8 mm
- net Net-(R43-Pad1): track 0.00 -> 4.49 mm
- net Net-(Q7-Pad1): track 4.32 -> 0.00 mm
- net Net-(D11-Pad2): track 10.7 -> 14.7 mm
- net Net-(Q4-Pad3): track 0.00 -> 3.30 mm
- net Net-(Q5-Pad3): track 4.54 -> 1.42 mm
- net Net-(Q6-Pad1): track 2.05 -> 5.07 mm
- net Net-(Q4-Pad2): track 2.99 -> 0.00 mm
- net /ADC12_IN9: track 41.6 -> 44.3 mm
- net Net-(Q1-Pad1): track 2.43 -> 0.00 mm
- net Net-(Q2-Pad1): track 2.41 -> 0.00 mm
- net Net-(P27-Pad4): track 4.29 -> 6.66 mm
- net /XA_12V: track 12.5 -> 14.8 mm
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Other:
- board text added: "Desgined by A.Mizuta in 2019/04/02."
- board text added: "STM32F407VGT6 Board "Centaurus" ver.1.1."
- board text removed: "Desgined by A.Mizuta in 2019/02/08."
- board text removed: "STM32F407VGT6 Board "Centaurus" ver.1.0."

Commit message: これで終わりであって欲しい.
Routing:
- net GND: vias 142 -> 299
Other:
- board text added: "3V3"
- board text added: "5V"
- board text added: "ADC"
- board text added: "H"
- board text added: "L"
- board text added: "OFF"
- board text added: "ON"
- board text added: "RX"
- board text added: "TX"
