File: Lipo-Alarm/Lipo_Alarm/Lipo_Alarm.kicad_pcb (KiCad board)
At the start: 2 copper layers, 50.5 x 34 mm, 79 parts, among them P1 SWD, P2 Cell_Check_Pin, P3 SERIAL0, Q1 NPN, SW1 RESET, SW2 SW0, SW3 SW1, U1 STM32F405RG, U2 AQM1602, U3 MC33063A, U4 MCP2221A, U5 LOGO, U6 Monster_Logo, X1 8MHz

Commit message: 一応、問題なさげ.
Parts:
- C1, C10, C11, C12, C13, C15, C2, C3, C4, C5, C6, C7, C8, C9: footprint Capacitors_SMD:C_0603 -> Mizz_lib:C_0603
- C16: footprint Capacitors_SMD:C_0805 -> Mizz_lib:C_0805
- C17: footprint Capacitors_SMD:C_0603 -> Mizz_lib:C_0805
- JP1: footprint Connect:GS2 -> Mizz_lib:GS2
- L1: value 22uH -> 220uH; footprint Mizz_lib:Inductor_Taiyo-Yuden_NR-50xx_HandSoldering -> Mizz_lib:Inductor_Taiyo-Yuden_NR-60xx_HandSoldering
- P3: footprint Mizz_lib:USB_Micro-B -> Mizz_lib:USB_Micro-B_Molex_47346-0001
- R1, R10, R11, R12, R13, R14, R15, R16, R17, R2, R20, R23, R24, R25, R26, R27, R28, R29, R3, R30, R4, R5, R6, R7, R8: footprint Resistors_SMD:R_0603 -> Mizz_lib:R_0603
- U3: footprint Housings_SOIC:SOIC-8_3.9x4.9mm_Pitch1.27mm -> Mizz_lib:SOIC-8_3.9x4.9mm_Pitch1.27mm
- U4: footprint Housings_SOIC:SOIC-14_3.9x8.7mm_Pitch1.27mm -> Mizz_lib:SOIC-14_3.9x8.7mm_Pitch1.27mm
- U5: footprint Mizz_lib:Battery_logo_7.0x7.0 -> Mizz_lib:Mini_Monster
- U6: value Monster_Logo -> LOGO; footprint Mizz_lib:Mini_Monster -> Mizz_lib:Battery_logo_7.0x7.0
- moved C14 0.79 mm to (125.0, 99.0)
- moved L1 0.57 mm to (126.0, 103.2)
- moved D4 0.50 mm to (117.8, 88.0)
- moved D7 0.50 mm to (117.8, 95.8)
- moved C1 0.36 mm to (130.5, 85.2)
- moved C3 0.28 mm to (128.0, 85.2)
- moved D11 0.25 mm to (131.2, 98.5)
- moved D3 0.25 mm to (117.8, 85.2)
- moved D5 0.25 mm to (117.8, 90.5)
- moved D6 0.25 mm to (117.8, 93.0)
- moved D1 0.11 mm to (150.2, 84.8)
- turned Q1 to 270 degrees
Connections:
- D1 pad 1: Net-(D1-Pad1) -> +3.3V
- D1 pad 2: +3.3V -> Net-(D1-Pad2)
- D11 pad 1: GND -> Net-(D11-Pad1)
- D11 pad 2: Net-(D11-Pad2) -> GND
- D2 pad 1: Net-(D2-Pad1) -> +3.3V
- D2 pad 2: +3.3V -> Net-(D2-Pad2)
- D3 pad 1: /1cell_batt -> +BATT
- D3 pad 2: +BATT -> /1cell_batt
- D4 pad 1: /2cell_batt -> +BATT
- D4 pad 2: +BATT -> /2cell_batt
- D5 pad 1: /3cell_batt -> +BATT
- D5 pad 2: +BATT -> /3cell_batt
- D6 pad 1: /4cell_batt -> +BATT
- D6 pad 2: +BATT -> /4cell_batt
- D7 pad 1: /5cell_batt -> +BATT
- D7 pad 2: +BATT -> /5cell_batt
- JP1 pad 1: Net-(D1-Pad1) -> Net-(D1-Pad2)
- L1 pad 2: Net-(D11-Pad2) -> Net-(D11-Pad1)
- Q1 pad 1: Net-(Q1-Pad1) -> GND
- Q1 pad 2: GND -> Net-(Q1-Pad2)
- Q1 pad 3: Net-(D2-Pad1) -> Net-(D2-Pad2)
- R6 pad 1: Net-(Q1-Pad1) -> Net-(Q1-Pad2)
- SP1 pad 2: Net-(D2-Pad1) -> Net-(D2-Pad2)
- U3 pad 2: Net-(D11-Pad2) -> Net-(D11-Pad1)
Routing:
- net Net-(D11-Pad1): track 0.00 -> 10.7 mm
- net Net-(D11-Pad2): track 10.6 -> 0.00 mm
- net Net-(D2-Pad1): track 8.46 -> 0.00 mm
- net Net-(D2-Pad2): track 0.00 -> 7.96 mm
- net Net-(Q1-Pad1): track 2.29 -> 0.00 mm
- net Net-(Q1-Pad2): track 0.00 -> 2.22 mm
- net Net-(D1-Pad2): track 0.00 -> 1.88 mm
- net Net-(D1-Pad1): track 1.88 -> 0.00 mm
- net /D-: track 10.5 -> 11.8 mm
- net /3cell_batt: track 4.42 -> 5.36 mm
- net /ADC12_IN0: track 19.5 -> 18.6 mm, vias 2 -> 1
- net GND: track 20.9 -> 21.4 mm, vias 324 -> 317
