File: Lipo-Alarm/Lipo_Alarm/Lipo_Alarm.sch (KiCad schematic (older format))
At the start: 78 parts, among them P1 SWD, P2 Cell_Check_Pin, P3 SERIAL0, Q1 NPN, SW1 RESET, SW2 SW0, SW3 SW1, U1 STM32F405RG, U2 AQM1602, U3 MC33063A, U4 MCP2221A, U5 LOGO, U6 Monster_Logo, X1 8MHz

Commit message: 一応、問題なさげ.
Parts:
- removed U2: AQM1602, Mizz_lib:AQM1602, symbol Hori_lib:AQM1602
- removed U5: LOGO, Mizz_lib:Battery_logo_7.0x7.0, symbol myDevice:LOGO
- removed U6: Monster_Logo, Mizz_lib:Mini_Monster, symbol Miz:Monster_Logo
- added U2: AQM1602, Mizz_lib:AQM1602, symbol Miz:AQM1602
- added U5: LOGO, Mizz_lib:Mini_Monster, symbol Miz:LOGO
- added U6: LOGO, Mizz_lib:Battery_logo_7.0x7.0, symbol Miz:LOGO
- C1, C10, C11, C12, C13, C15, C2, C3, C4, C5, C6, C7, C8, C9: footprint Capacitors_SMD:C_0603 -> Mizz_lib:C_0603
- C16: footprint Capacitors_SMD:C_0805 -> Mizz_lib:C_0805
- C17: footprint Capacitors_SMD:C_0603 -> Mizz_lib:C_0805
- JP1: footprint Connect:GS2 -> Mizz_lib:GS2
- L1: value 22uH -> 220uH; footprint Mizz_lib:Inductor_Taiyo-Yuden_NR-50xx_HandSoldering -> Mizz_lib:Inductor_Taiyo-Yuden_NR-60xx_HandSoldering
- P3: footprint Mizz_lib:USB_Micro-B -> Mizz_lib:USB_Micro-B_Molex_47346-0001
- R1, R10, R11, R12, R13, R14, R15, R16, R17, R2, R20, R23, R24, R25, R26, R27, R28, R29, R3, R30, R4, R5, R6, R7, R8: footprint Resistors_SMD:R_0603 -> Mizz_lib:R_0603
- U3: footprint Housings_SOIC:SOIC-8_3.9x4.9mm_Pitch1.27mm -> Mizz_lib:SOIC-8_3.9x4.9mm_Pitch1.27mm
- U4: footprint Housings_SOIC:SOIC-14_3.9x8.7mm_Pitch1.27mm -> Mizz_lib:SOIC-14_3.9x8.7mm_Pitch1.27mm
