File: Parent_Turtle_RC19ver5.1.1kran_main_ver/Parent_Turtle_RC19main.sch (KiCad schematic (older format))
At the start: 81 parts, among them P1 CONN_02X15, P10 WRITING, P11 ADC, P12 5V_in, P13 ADC/Vdd/GND, P14 I/O, P15 I/O /Vdd/GND, P16 PWM, P17 SERIAL1, P19 ENC3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

Commit message: パク君のシールドmain基板.
Connections:
- net E10: no longer P16.4 (P4)
- net E11: now also P16.4 (P4)
Other:
- note removed: "<- currern is very low."
- note removed: "http://akizukidenshi.com/catalog/g/gP-06984/"
Changed lines of the file:
@@
 	1    0    0    -1
 $EndComp
-Text Notes 5700 700  0    60   ~ 0
-http://akizukidenshi.com/catalog/g/gP-06984/
 Text Label 8925 4925 0    60   ~ 0
 C6
@@
 Wire Wire Line
 	4925 650  4925 950
-Text Notes 8050 700  0    60   ~ 0
-<- currern is very low.
 Text Label 7750 3800 2    60   ~ 0
 A2
@@
 E9
 Text Label 4125 4550 2    60   ~ 0
-E10
+E11
 $Comp
 L conn:CONN_02X04 P5
