File: Parent_Turtle_RC19ver5.1.1kran_main_ver/Parent_Turtle_RC19main.kicad_pcb (KiCad board)
At the start: 2 copper layers, 70 x 60 mm, 81 parts, among them P1 CONN_02X15, P10 WRITING, P11 ADC, P12 5V_in, P13 ADC/Vdd/GND, P14 I/O, P15 I/O /Vdd/GND, P16 PWM, P17 SERIAL1, P19 ENC3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

Commit message: パク君のシールドmain基板.
Connections:
- P16 pad 4: /E10 -> /E11
Routing:
- net /E10: track 8.60 -> 0.00 mm
- net /E11: track 0.75 -> 6.02 mm
Changed lines of the file:
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@@
     (thickness 1.6)
     (drawings 13)
-    (tracks 522)
+    (tracks 520)
     (zones 0)
     (modules 81)
@@
   )
   (setup
-    (last_trace_width 0.5)
+    (last_trace_width 0.3)
     (user_trace_width 0.3)
     (user_trace_width 0.5)
@@
       (net 24 /E9))
     (pad 4 thru_hole oval (at 0 7.62) (size 1.7 1.7) (drill 1) (layers *.Cu *.Mask)
-      (net 27 /E10))
+      (net 26 /E11))
     (model ${KISYS3DMOD}/Connector_PinHeader_2.54mm.3dshapes/PinHeader_1x04_P2.54mm_Vertical.wrl
       (at (xyz 0 0 0))
@@
   (segment (start 152.55 127) (end 152.55 128.1) (width 0.5) (layer B.Cu) (net 1))
   (segment (start 152.55 128.1) (end 152.93 128.48) (width 0.5) (layer B.Cu) (net 1))
-  (segment (start 127.6002 122.55068) (end 127.6002 122.9402) (width 0.5) (layer B.Cu) (net 104))
   (segment (start 150.27 127) (end 152.55 127) (width 0.5) (layer B.Cu) (net 1))
   (segment (start 152.55 125.3) (end 152 124.75) (width 0.5) (layer B.Cu) (net 1))
@@
   (segment (start 115.715 107.435) (end 115.695 107.435) (width 0.3) (layer B.Cu) (net 25))
   (segment (start 113.175 109.975) (end 112.425 109.975) (width 0.3) (layer B.Cu) (net 26))
-  (segment (start 108.909999 108.760001) (end 108.06 109.61) (width 0.3) (layer B.Cu) (net 27))
-  (segment (start 109.021399 108.648601) (end 108.909999 108.760001) (width 0.3) (layer B.Cu) (net 27))
-  (segment (start 114.388601 108.648601) (end 109.021399 108.648601) (width 0.3) (layer B.Cu) (net 27))
-  (segment (start 115.715 109.975) (end 114.388601 108.648601) (width 0.3) (layer B.Cu) (net 27))
+  (segment (start 108.425 109.975) (end 108.06 109.61) (width 0.3) (layer B.Cu) (net 26))
+  (segment (start 113.175 109.975) (end 108.425 109.975) (width 0.3) (layer B.Cu) (net 26))
   (segment (start 114.388601 118.177529) (end 113.18613 119.38) (width 0.3) (layer B.Cu) (net 30))
   (segment (start 113.175 115.055) (end 114.388601 116.268601) (width 0.3) (layer B.Cu) (net 30))
@@
   (segment (start 128.49 105.27) (end 128.485 105.265) (width 0.3) (layer B.Cu) (net 103))
   (segment (start 128.49 107.71) (end 128.49 105.27) (width 0.3) (layer B.Cu) (net 103))
+  (segment (start 127.6002 122.55068) (end 127.6002 122.9402) (width 0.5) (layer B.Cu) (net 104))
   (zone (net 2) (net_name GND) (layer B.Cu) (hatch edge 0.508)
     (connect_pads yes (clearance 0.2))
@@
       )
     )
+  )
+  (zone (net 0) (net_name "") (layer B.Cu) (hatch edge 0.508)
+    (connect_pads (clearance 0.2))
+    (min_thickness 0.254)
+    (keepout (tracks allowed) (vias allowed) (copperpour not_allowed))
+    (fill (arc_segments 16) (thermal_gap 0.508) (thermal_bridge_width 0.508))
+    (polygon
+      (pts
+        (xy 164.56 108.99) (xy 164.56 113.99) (xy 169.31 113.99) (xy 169.31 108.99)
+      )
+    )

Commit message: mainは加工データを追加,電源はビアホールなどの配線の改良.
Parts:
- moved U4 2.44 mm to (128.2, 98.9)

Commit message: ステンシル自作実験台ファイルを生成した
Parts:
- removed U4: LOGO, Mizz_lib:Turtle_Logo_15.0x15.0
