File: POWER/Electrocity Manager/Electrocity Manager.sch (KiCad schematic (older format))
At the start: 47 parts

Commit message: 電源、上がっていなかったやつ
Parts:
- removed C? (x12): C, symbol device:C
- removed C? (x2): 2.2u, symbol device:C
- removed C? (x2): 22p, symbol device:C
- removed D?: 12V, symbol device:LED
- removed D?: 5V, symbol device:LED
- removed D?: 3.3V, symbol device:LED
- removed D?: BATT, symbol device:LED
- removed D?: POWER_OUT, symbol device:LED
- removed D?: SENSERD, symbol device:LED
- removed D?: DIODE, symbol device:DIODE
- removed JP?: 3.3V_JP, symbol device:JUMPER
- removed P? (x2): BATT_IN, symbol conn:CONN_01X02
- removed P?: SWD, symbol conn:CONN_01X06
- removed R? (x3): 2.4k, symbol device:R
- removed R? (x2): R, symbol device:R
- removed R?: 10k, symbol device:R
- removed R?: R_JP, symbol device:R
- removed U?: STM32F405RG_excerpt, LQFP64, symbol stm32f405rg_excerpt:STM32F405RG_excerpt
- removed U?: CCG30-24-05S, symbol Miz:CCG30-24-xxS
- removed U?: CCG30-24-12S, symbol Miz:CCG30-24-xxS
- removed U? (x2): ACS781, symbol Miz:ACS781
- removed U? (x2): RELAY, symbol Miz:RELAY
- removed U? (x2): TLP291, Package_DIP:SMDIP-4_W7.62mm, symbol Isolator:TLP291
- removed U?: AZ1086H, symbol myDevice:AZ1086H
- removed U?: LOGO, symbol myDevice:LOGO
- removed U?: MAX3051, symbol Interface_UART:MAX3051
- removed X?: CRYSTAL, symbol device:CRYSTAL
- added C?: 4.7u, symbol device:C
- added C? (x21): 0.1u, symbol device:C
- added C? (x3): 1u, symbol device:C
- added C?: 10u, symbol device:C
- added C? (x2): 22u, symbol device:C
- added C? (x2): 2.2u, symbol device:C
- added C? (x2): 22p, symbol device:C
- added C?: C, symbol device:C
- added C?: 470p, symbol device:C
- added C?: 100u, symbol device:C
- added C? (x2): 470u, symbol device:CP1
- added D? (x10): DIODE, symbol device:DIODE
- added D? (x3): LED, symbol device:LED
- added D?: LED0, symbol device:LED
- added D?: LED1, symbol device:LED
- added D?: LED2, symbol device:LED
- added D?: LED3, symbol device:LED
- added D?: LED4, symbol device:LED
- added D?: BATT, symbol device:LED
- added D?: Main_POWER, symbol device:LED
- added D? (x2): Relay_BATT, symbol device:LED
- added IC? (x2): TLP291, SOP4, symbol opto:TLP291
- added JP?: 3.3V_JP, symbol device:JUMPER
- added JP?: CAN0_JP, symbol device:JUMPER
- added JP?: Relay_JP, symbol device:JUMPER
- added L?: 22uH, symbol device:INDUCTOR_SMALL
- added L?: 22u, symbol device:INDUCTOR_SMALL
- added P? (x2): CAN0, symbol conn:CONN_01X04
- added P?: SWD, symbol conn:CONN_01X06
- added P? (x2): BATT_IN, symbol conn:CONN_01X02
- added P?: POWER_OUT, symbol conn:CONN_01X02
- added P?: FUN_OUT, symbol conn:CONN_01X02
- added P?: FRAME_GND, symbol conn:CONN_01X01
- added P?: Main_SW, symbol conn:CONN_01X02
- added P? (x2): EMERGENCY, symbol conn:CONN_01X02
- added P?: SERIAL0, symbol conn:CONN_01X04
- added P? (x2): 12V_Out, symbol conn:CONN_01X02
- added P? (x2): main_12V_Out, symbol conn:CONN_01X04
- added P? (x2): 5V_Out, symbol conn:CONN_01X02
- added Q?: NPN, symbol device:NPN
- added Q? (x2): MOSFET_N, symbol device:MOSFET_N
- added R? (x9): 10k, symbol device:R
- added R?: R_JP, symbol device:R
- added R?: 120, symbol device:R
- added R?: 1.2k, symbol device:R
- added R? (x2): 510, symbol device:R
- added R? (x10): 330, symbol device:R
- added R? (x4): 10, symbol device:R
- added R? (x4): R, symbol device:R
- added R?: 4.7, symbol device:R
- added R? (x3): 2.2k, symbol device:R
- added R? (x2): 4.7k, symbol device:R
- added R?: 50k, symbol device:R
- added R?: 1.3k, symbol device:R
- added R?: 160, symbol device:R
- added SP?: SPEAKER, symbol device:SPEAKER
- added SW?: SW0, symbol device:SW_PUSH
- added SW?: SW1, symbol device:SW_PUSH
- added SW?: SW2, symbol device:SW_PUSH
- added SW?: RESET, symbol device:SW_PUSH
- added U?: STM32F405RG, Housings_QFP:LQFP-44_10x10mm_Pitch0.8mm, symbol stm32f405rg_excerpt:STM32F405RG_excerpt
- added U?: AZ1086H, symbol myDevice:AZ1086H
- added U?: MAX3051, symbol myDevice:MAX3051
- added U?: CCG30-24-12S, symbol Miz:CCG30-24-xxS
- added U?: OSTBABS4C2B, symbol myDevice:OSTBABS4C2B
- added U? (x3): ACS781, symbol Miz:ACS781
- added U?: AQM1602_BL, symbol Miz:AQM1602_BL
- added U?: MC33063A, symbol Miz:MC33063A
- added U? (x2): RELAY, symbol Hori_lib:RELAY
- added U?: BD9G101G, symbol myDevice:BD9G101G
- added X?: 8MHz, symbol device:CRYSTAL
Connections:
- net labels added: +12P, 12V_Current_Out, 24V, ADC12_INx, CAN1_RX, CAN1_TX, Coil_IN, CurrentSensor_IN0, CurrentSensor_IN1, FB, Force_Shutdown, I2C_SCL, I2C_SDA, Main_Power, PXx, Relay_Out, Relay_State, TIMx_CHx, To_Fun, To_MD, To_RelayB, USARTx_RX, USARTx_TX, Voltage_Divide, ~NRST
- net labels removed: CAN0_RX, CAN0_TX, Current_Sensor0, Current_Sensor1, NRST, Senserd
- wire segments 57 -> 302
- no-connect marks 2 -> 6
