File: サーボ用電源基板/サーボ用電源基板_絶対制御電源＆パワー系落とすマン/サーボ用電源基板_12Vout_BattOut.sch (KiCad schematic (older format))
At the start: 57 parts, among them IC1 TLP291, IC2 TLP291, P1 BATT_IN, P10 MAIN_SW, P2 BATT_IN, P3 OUT_A, P4 OUT_B, P5 EMERGENCY_SIGNAL, P6 12V, P7 12V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

Commit message: 恐らくエネルギー破壊で燃えた
Parts:
- removed C10, C11: 47u, Capacitor_THT:CP_Radial_D4.0mm_P2.00mm, symbol device:CP1
- removed C6, C7: 0.1u, Capacitors_SMD:C_0603, symbol device:C
- removed C8, C9: 10u, Capacitors_ThroughHole:C_Disc_D6_P5, symbol device:C
- removed D7: OUT_B, LED_THT:LED_D3.0mm_Clear, symbol device:LED
- removed D8, D9: DIODESCH, Diode_SMD:D_PowerDI-123, symbol device:DIODESCH
- removed L1, L2: 10uH, Inductor_SMD:L_Vishay_IHLP-6767, symbol device:INDUCTOR_SMALL
- removed R11: 1k, Resistor_SMD:R_0603_1608Metric, symbol device:R
- removed R12, R14: 10k, Resistor_SMD:R_0603_1608Metric, symbol device:R
- removed R13, R15: 2.2k, Resistor_SMD:R_0603_1608Metric, symbol device:R
- removed U3, U4: RT8289, Package_SO:SOIC-8-1EP_3.9x4.9mm_P1.27mm_EP2.29x3mm_ThermalVias, symbol Miz:RT8289
Connections:
- net labels added: Power_OUT
- net labels removed: 7V_OUTA, 7V_OUTB, DCDC_BATT, FB_A, FB_B
- wire segments 101 -> 56
- no-connect marks 8 -> 2
Other:
- moved on the sheet: D2, D3, D4, D6, R10, R6, R7, R8
