File: stm32f4_Centaurus_ver.1.1/stm32f4_Centaurus/stm32f4_Centaurus.kicad_pcb (KiCad board)
At the start: 2 copper layers, 100 x 79 mm, 207 parts, among them IC1 PIC24FJ64GB004, P1 PICKit3, P10 XA2_12V, P11 CAN0, P12 CAN1, P13 CAN0, P14 CAN1, P15 SERIAL2, P16 SERIAL0, P17 XA2_5V, P18 SWD, P2 SERIAL5_SBDBT, P23 A/D, P24 PWM, P25 A/D_batt, P26 PWM_batt, P27 EMERGENCY_CHECK, P28 I/O_5V, P29 I/O_Variable, P3 ENC0, P30 I/O_5V_batt, P31 I/O_Variable, P4 ENC2, P5 SERIAL1, P6 ENC3, P7 ENC1, P8 SERIAL4, P9 SERIAL3, Q1 FET_P, Q2 FET_P, Q3 FET_P, Q4 NPN, Q5 NPN, Q6 FET_P, Q7 FET_N, SW1 Main_POWER, SW2 SW1, SW3 SW0, SW4 SW2, SW5 SW3, U1 STM32F407VG, U10 LOGO, U12 25LC010A, U13 LOGO, U2 AZ1086H, U3 MCP2221A, U4 AP3211, U5 MAX3051, U6 MAX3051, U7 AQM1602_BL, U8 OSTBABS4C2B, U9 LOGO, X1 8MHz

Commit message: 完成.
Other:
- board text added: "D+"
- board text added: "D-"
Changed lines of the file:
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@@
   (general
     (thickness 1.6)
-    (drawings 129)
+    (drawings 133)
     (tracks 2630)
     (zones 0)
@@
     (47 F.CrtYd user)
     (48 B.Fab user)
-    (49 F.Fab user)
+    (49 F.Fab user hide)
   )
   (setup
@@
     )
   )
+  (gr_text 5V (at 132 126.75) (layer B.SilkS)
+    (effects (font (size 0.8 0.8) (thickness 0.2)) (justify mirror))
+  )
+  (gr_text D- (at 134.55 126.75) (layer B.SilkS)
+    (effects (font (size 0.8 0.8) (thickness 0.2)) (justify mirror))
+  )
+  (gr_text D+ (at 136.55 126.75) (layer B.SilkS)
+    (effects (font (size 0.8 0.8) (thickness 0.2)) (justify mirror))
+  )
+  (gr_text GND (at 139.15 126.75) (layer B.SilkS)
+    (effects (font (size 0.8 0.8) (thickness 0.2)) (justify mirror))
+  )
   (gr_text 5V (at 144.25 59.75) (layer F.SilkS)
     (effects (font (size 0.8 0.8) (thickness 0.2)))
@@
   (via (at 102.75 79) (size 0.8) (drill 0.4) (layers F.Cu B.Cu) (net 2))
   (via (at 84.75 79) (size 0.8) (drill 0.4) (layers F.Cu B.Cu) (net 2))
-  (via (at 75.75 68.25) (size 0.8) (drill 0.4) (layers F.Cu B.Cu) (net 2))
+  (via (at 75.75 69.25) (size 0.8) (drill 0.4) (layers F.Cu B.Cu) (net 2))
   (via (at 86 65.5) (size 0.8) (drill 0.4) (layers F.Cu B.Cu) (net 2))
   (via (at 90.5 71.5) (size 0.8) (drill 0.4) (layers F.Cu B.Cu) (net 2))
