File: 実験用電源基板/Power_exp/Power_exp.kicad_pcb (KiCad board)
At the start: 2 copper layers, 80 x 55 mm, 43 parts, among them IC1 TLP291, IC2 TLP291, P1 EMERGENCY, P10 POWER_OUT, P11 FUN_OUT, P2 EMERGENCY, P3 POW_SW, P4 12v, P5 12v, P6 POWER_IN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

Commit message: 完成（仮）
Parts:
- moved P7 56.4 mm to (147.8, 55.2)
- moved C3 50.9 mm to (156.2, 104.2), turned to 90 degrees
- moved P1 42.5 mm to (138.0, 102.1), turned to 0 degrees
- moved D7 42.0 mm to (131.2, 55.5), turned to 180 degrees
- moved P10 40.2 mm to (129.9, 94.4)
- moved D6 40.2 mm to (130.9, 88.0)
- moved R11 40.2 mm to (132.8, 90.0)
- moved R12 38.8 mm to (132.8, 57.1), turned to 135 degrees
- moved P2 37.8 mm to (145.5, 102.1), turned to 0 degrees
- moved P11 37.8 mm to (130.0, 62.0), turned to 0 degrees
- moved P5 36.8 mm to (194.2, 86.0), turned to 90 degrees
- moved C2 35.4 mm to (196.5, 77.2), turned to 90 degrees
- moved C5 35.3 mm to (193.0, 67.5), turned to 90 degrees
- moved P4 35.3 mm to (194.2, 78.5), turned to 90 degrees
- moved C1 33.4 mm to (192.1, 84.8), turned to 90 degrees
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Routing:
- net /24v: track 0.00 -> 75.5 mm
- net +BATT: track 0.00 -> 35.3 mm
- net /Coil: track 0.50 -> 35.5 mm
- net /Coil_Out: track 0.00 -> 22.4 mm
- net /Relay_state: track 19.5 -> 37.2 mm
- net Net-(IC1-Pad3): track 0.00 -> 11.9 mm
- net /RelayA_Coil_In: track 0.00 -> 5.50 mm
- net Net-(JP1-Pad1): track 0.00 -> 5.44 mm
- net /Forced_shutdown: track 10.7 -> 16.0 mm
- net Net-(P1-Pad1): track 0.00 -> 5.00 mm
- net /Fun_Out: track 0.00 -> 4.31 mm
- net Net-(D1-Pad2): track 0.00 -> 4.22 mm
- net +12V: track 86.4 -> 83.5 mm
- net Net-(D3-Pad1): track 0.00 -> 2.22 mm
- net Net-(IC1-Pad1): track 0.00 -> 2.11 mm
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- added copper zone on B.Cu, net +BATT
- added copper zone on B.Cu, net /Fun_Out
- added copper zone on B.Cu, net /Power_Out
Other:
- outline, holes or cut-outs redrawn

Commit message: 実験用電源基板(うちで加工する用)
Parts:
- D1: footprint Mizz_lib:SOD-123 -> Diodes_SMD:SMB_Handsoldering
- moved D6 15.7 mm to (128.2, 72.5)
- moved P10 15.7 mm to (127.2, 78.9)
- moved R11 15.7 mm to (130.0, 74.5)
- moved U3 14.8 mm to (156.0, 71.0), turned to 90 degrees
- moved D2 14.8 mm to (128.2, 85.2)
- moved R7 14.8 mm to (130.0, 86.8)
- moved P6 14.8 mm to (127.2, 91.4)
- moved P7 14.2 mm to (133.5, 55.2)
- moved U2 8.39 mm to (140.8, 71.0), turned to 90 degrees
- moved D1 7.84 mm to (134.5, 96.2)
- moved JP1 5.55 mm to (168.0, 56.5), turned to 270 degrees
- moved D7 5.20 mm to (128.2, 59.8)
- moved P11 5.20 mm to (127.0, 66.2)
- moved R12 5.20 mm to (129.8, 61.4)
- moved R3 3.16 mm to (167.7, 64.5), turned to 0 degrees
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Connections:
- JP1 pad 1: Net-(JP1-Pad1) -> GNDPWR
- Q1 pad 2: /Coil_Out -> GNDPWR
- Q1 pad 3: Net-(JP1-Pad1) -> /Coil_Out
- R3 pad 2: Net-(JP1-Pad1) -> GNDPWR
- U2 pad 1: /RelayA_Coil_In -> /Coil
- U3 pad 2: /RelayA_Coil_In -> /Coil_Out
Routing:
- net /Coil_Out: track 22.4 -> 51.4 mm
- net +BATT: track 35.3 -> 7.29 mm
- net /Coil: track 35.5 -> 63.4 mm
- net Net-(IC1-Pad3): track 11.9 -> 5.88 mm
- net /RelayA_Coil_In: track 5.50 -> 0.00 mm
- net Net-(JP1-Pad1): track 5.44 -> 0.00 mm
- net +12V: track 83.5 -> 78.5 mm
- net /24v: track 75.5 -> 78.3 mm
- net /Forced_shutdown: track 16.0 -> 14.7 mm
- net Net-(IC1-Pad1): track 2.11 -> 3.13 mm
- net Net-(D3-Pad1): track 2.22 -> 1.68 mm
Other:
- outline, holes or cut-outs redrawn
