File: 実験用電源基板/Power_exp/Power_exp.sch (KiCad schematic (older format))
At the start: 12 parts

Commit message: 一旦挙げておく.
Parts:
- added C1, C2, C4, C5: 0.1u, Capacitors_SMD:C_0603, symbol device:C
- added C3, C6: 470, Capacitors_ThroughHole:C_Radial_D10_L20_P5, symbol device:CP1
- added D1: DIODE, Mizz_lib:SOD-123, symbol device:DIODE
- added D6, D7: LED, LEDs:LED-3MM, symbol device:LED
- added IC1, IC2: TLP291, Housings_DIP:DIP-4_W7.62mm, symbol opto:TLP291
- added JP1: JUMPER, Pin_Headers:Pin_Header_Straight_1x02, symbol device:JUMPER
- added P1, P2: EMERGENCY, RP_KiCAD_Connector:XA_2T, symbol conn:CONN_01X02
- added P10: POWER_OUT, RP_KiCAD_Connector:XT60_T, symbol conn:CONN_01X02
- added P11: FUN_OUT, RP_KiCAD_Connector:XT60_T, symbol conn:CONN_01X02
- added P3: POW_SW, RP_KiCAD_Connector:XA_2T, symbol conn:CONN_01X02
- added P4, P5: 12v, RP_KiCAD_Connector:XA_2T, symbol conn:CONN_01X02
- added P8: main-signal, RP_KiCAD_Connector:XA_4T, symbol conn:CONN_01X04
- added P9: main-signal, RP_KiCAD_Connector:XA_4L, symbol conn:CONN_01X04
- added Q1: MOSFET_N_123, TO_SOT_Packages_SMD:SOT-23_Handsoldering, symbol Hori_lib:MOSFET_N_123
- added R1, R3, R5: 2.2k, Resistors_SMD:R_0603, symbol device:R
- added R11, R12, R2: 4.7k, Resistors_SMD:R_0603, symbol device:R
- added R4: 330, Resistors_SMD:R_0603, symbol device:R
- added R6: 10k, Resistors_SMD:R_0603, symbol device:R
- added U1: CCG30-24-xxS, Mizz_lib:CCG30-24-xxS, symbol Miz:CCG30-24-xxS
- D2, D3, D4, D5: renamed from D?; footprint (none) -> LEDs:LED-3MM
- P6: renamed from P?; value BATT1 -> POWER_IN; footprint (none) -> RP_KiCAD_Connector:XT60_T
- P7: renamed from P?; value GND1 -> FRAMEGND; footprint (none) -> Wire_Pads:SolderWirePad_single_2mmDrill
- R10, R7, R8: renamed from R?; value R -> 4.7k; footprint (none) -> Resistors_SMD:R_0603
- R9: renamed from R?; value R -> 2.2k; footprint (none) -> Resistors_SMD:R_0603
- U2, U3: renamed from U?; footprint (none) -> Mizz_lib:V23074A2002A403
Connections:
- net labels added: Coil_Out, Forced_shutdown, Fun_Out, Power_Out, RelayA_Coil_In, Relay_state
- wire segments 0 -> 73
- no-connect marks 0 -> 3
Other:
- note added: "main to power signal about Emergency."
- moved on the sheet: D2, D3, D4, D5, P6, P7, R10, R7, R8, R9

Commit message: 実験用電源基板(うちで加工する用)
Parts:
- D1: footprint Mizz_lib:SOD-123 -> Diodes_SMD:SMB_Handsoldering
Connections:
- net labels removed: RelayA_Coil_In
Changed lines of the file:
@@
 24v
-$Comp
-L device:DIODE D1
-U 1 1 5C5F96CC
-P 4025 1675
-F 0 "D1" H 4025 1483 40  0000 C CNN
-F 1 "DIODE" H 4025 1559 40  0000 C CNN
-F 2 "Mizz_lib:SOD-123" H 4025 1675 60  0001 C CNN
-F 3 "" H 4025 1675 60  0000 C CNN
-	1    4025 1675
-	-1   0    0    1
-$EndComp
 $Comp
 L power:+BATT #PWR07
@@
 F 3 "" H 3320 5050 60  0000 C CNN
 	1    3225 5050
-	-1   0    0    1
+	-1   0    0    -1
 $EndComp
 $Comp
@@
 Text Label 7050 3825 0    50   ~ 0
 Fun_Out
-Text Label 7700 2950 0    50   ~ 0
-RelayA_Coil_In
-Text Label 7700 4500 0    50   ~ 0
-RelayA_Coil_In
-Wire Wire Line
-	7700 4500 7675 4500
 $Comp
 L conn:CONN_01X02 P2
@@
 Text Label 6550 1525 1    50   ~ 0
 Fun_Out
+$Comp
+L power:GNDPWR #PWR0103
+U 1 1 5C67851B
+P 2600 5400
+F 0 "#PWR0103" H 2600 5450 40  0001 C CNN
+F 1 "GNDPWR" H 2595 5468 40  0000 C CNN
+F 2 "" H 2600 5400 60  0000 C CNN
+F 3 "" H 2600 5400 60  0000 C CNN
+	1    2600 5400
+	1    0    0    -1
+$EndComp
+Wire Bus Line
+	6450 6100 6425 6225
+Wire Wire Line
+	2600 5400 2600 5375
+Connection ~ 2600 5375
+Text Label 7675 4500 0    50   ~ 0
+Coil
+Text Label 7700 2950 0    50   ~ 0
+Coil_Out
+$Comp
+L device:DIODE D1
+U 1 1 5C70781D
+P 4025 1675
+F 0 "D1" H 4025 1483 40  0000 C CNN
+F 1 "DIODE" H 4025 1559 40  0000 C CNN
+F 2 "Diodes_SMD:SMB_Handsoldering" H 4025 1675 60  0001 C CNN
+F 3 "" H 4025 1675 60  0000 C CNN
+	1    4025 1675
+	-1   0    0    1
+$EndComp
 $EndSCHEMATC

Commit message: 資料のコス用の基板外形サイズなどの出力.
Parts:
- D1: symbol device:DIODE -> Power_exp-rescue:DIODE-device
- Q1: symbol Hori_lib:MOSFET_N_123 -> Power_exp-rescue:MOSFET_N_123-Hori_lib
- U2, U3: symbol V23074A2002A403:V23074A2002A403 -> Power_exp-rescue:V23074A2002A403-V23074A2002A403
Changed lines of the file:
@@
 $EndDescr
 $Comp
-L V23074A2002A403:V23074A2002A403 U3
+L Power_exp-rescue:V23074A2002A403-V23074A2002A403 U3
 U 1 1 5C55B9A1
 P 7150 3150
@@
 $EndComp
 $Comp
-L V23074A2002A403:V23074A2002A403 U2
+L Power_exp-rescue:V23074A2002A403-V23074A2002A403 U2
 U 1 1 5C55B9E7
 P 7125 4300
@@
 F 1 "TLP291" H 4000 5332 40  0000 C CNN
 F 2 "Housings_DIP:DIP-4_W7.62mm" H 4000 5265 29  0000 C CNN
-F 3 "http://www.semicon.toshiba.co.jp/docs/datasheet/en/Opto/TLP291_en_datasheet_120426.pdf" H 4000 5182 60  0000 C CNN
+F 3 "http://www.semicon.toshiba.co.jp/docs/datasheet/en/Opto/TLP291_en_datasheet_120426.pdf" H 4000 5182 60  0001 C CNN
 	1    4000 4950
 	-1   0    0    -1
@@
 F 1 "TLP291" H 4000 6507 40  0000 C CNN
 F 2 "Housings_DIP:DIP-4_W7.62mm" H 4000 6440 29  0000 C CNN
-F 3 "http://www.semicon.toshiba.co.jp/docs/datasheet/en/Opto/TLP291_en_datasheet_120426.pdf" H 4000 6357 60  0000 C CNN
+F 3 "http://www.semicon.toshiba.co.jp/docs/datasheet/en/Opto/TLP291_en_datasheet_120426.pdf" H 4000 6357 60  0001 C CNN
 	1    4000 6125
 	1    0    0    -1
@@
 $EndComp
 $Comp
-L Hori_lib:MOSFET_N_123 Q1
+L Power_exp-rescue:MOSFET_N_123-Hori_lib Q1
 U 1 1 5C62A97B
 P 3225 5050
@@
 Coil_Out
 $Comp
-L device:DIODE D1
+L Power_exp-rescue:DIODE-device D1
 U 1 1 5C70781D
 P 4025 1675
