File: Electrocity_Manager_Pikachu/Electrocity_Manager/Electrocity_Manager.sch (KiCad schematic (older format))
At the start: 190 parts, among them IC1 POW_ON, IC2 MAIN_SHUTDOWN, IC3 RELAY_STATE, IC4 ADC_RST, J1 SERIAL, P1 SWD, P10 EMERGENCY, P11 EMERGENCY, P12 FRAME_GRAND, P13 BATT_IN, P14 POWER_OUT, P15 FUN_OUT, P16 BATT_IN, P17 POWER_OUT, P18 FUN_OUT, P2 CAN, P3 CAN, P4 EMERGENCY_SIGNAL, P5 EMERGENCY_SIGNAL, P6 12V_OUT, P7 12V_OUT, P9 MAIN_SW, Q1 FET_N, Q2 NPN, Q3 NPN, Q7 FET_N, SW1 RST, SW2 SW0, SW3 SW1, U1 MAX3051, U10 NJM7812, U11 ACS781, U12 V23134J1052D642, U13 ACS70331, U14 ACS781, U15 BD33FA1, U16 LOGO, U17 LOGO, U18 LOGO, U19 MCP2221A, U2 STM32F405RG, U20 OSRB38C9AA, U21 OSRB38C9AA, U22 HSIN_946, U23 LOGO, U24 LOGO, U25 LOGO, U26 LOGO, U3 FULL COLOR, U4 AQM0802_BL, U5 AP3211, U6 SI8900, U7 AZ1086H, U8 V23134J1052D642, U9 RPA60-12FW/N, X1 8MHz

Commit message: ピカチュウたちの配線を変えた。
Parts:
- added U27: LOGO, Mizz_lib:kitLogo_Mask_5.0x5.0, symbol Electrocity_Manager-rescue:LOGO-myDevice
- added U28: LOGO, Mizz_lib:RedBull_Logo_Silk_16x16, symbol Electrocity_Manager-rescue:LOGO-myDevice
- C30, C31: footprint Mizz_lib:C_0603 -> Capacitors_SMD:C_0805
Changed lines of the file:
@@
 F 0 "C31" H 13750 5950 40  0000 L CNN
 F 1 "22u" H 13750 5800 40  0000 L CNN
-F 2 "Mizz_lib:C_0603" H 13788 5725 30  0001 C CNN
+F 2 "Capacitors_SMD:C_0805" H 13788 5725 30  0001 C CNN
 F 3 "" H 13750 5875 60  0000 C CNN
 	1    13750 5875
@@
 F 0 "C30" H 12900 5950 40  0000 L CNN
 F 1 "10u" H 12900 5800 40  0000 L CNN
-F 2 "Mizz_lib:C_0603" H 12938 5725 30  0001 C CNN
+F 2 "Capacitors_SMD:C_0805" H 12938 5725 30  0001 C CNN
 F 3 "" H 12900 5875 60  0000 C CNN
 	1    12900 5875
@@
 	15500 8625 15500 8525
 Connection ~ 15500 8625
+$Comp
+L Electrocity_Manager-rescue:LOGO-myDevice U27
+U 1 1 5CD86A01
+P 15525 4900
+F 0 "U27" H 15803 4953 60  0000 L CNN
+F 1 "LOGO" H 15803 4847 60  0000 L CNN
+F 2 "Mizz_lib:kitLogo_Mask_5.0x5.0" H 15525 4900 60  0001 C CNN
+F 3 "" H 15525 4900 60  0000 C CNN
+	1    15525 4900
+	1    0    0    -1
+$EndComp
+$Comp
+L Electrocity_Manager-rescue:LOGO-myDevice U28
+U 1 1 5CD88407
+P 15525 5500
+F 0 "U28" H 15803 5553 60  0000 L CNN
+F 1 "LOGO" H 15803 5447 60  0000 L CNN
+F 2 "Mizz_lib:RedBull_Logo_Silk_16x16" H 15525 5500 60  0001 C CNN
+F 3 "" H 15525 5500 60  0000 C CNN
+	1    15525 5500
+	1    0    0    -1
+$EndComp
 $EndSCHEMATC

Commit message: ピカチュウ.
Parts:
- D10: footprint TO_SOT_Packages_SMD:TO-277A -> Package_TO_SOT_SMD:TO-277B
Changed lines of the file:
@@
 F 0 "D10" H 8225 1975 50  0000 C CNN
 F 1 "SBR_DIODE" H 8225 1884 50  0000 C CNN
-F 2 "TO_SOT_Packages_SMD:TO-277A" H 8125 1650 50  0001 C CNN
+F 2 "Package_TO_SOT_SMD:TO-277B" H 8125 1650 50  0001 C CNN
 F 3 "" H 8125 1650 50  0001 C CNN
 	1    8225 1650
