File: フォトインタラプタ_隙間大きい/Phote_Big/Phote_Big.sch (KiCad schematic (older format))
At the start: 4 parts, among them P1 I/O connector, U1 LBT-131

Commit message: そういえば，RC19の基板整理していなかった(リポジトリ的にも)
Parts:
- R1: value 120 -> 240
Changed lines of the file:
@@
 EESchema Schematic File Version 4
 LIBS:Phote_Big-cache
-EELAYER 26 0
+EELAYER 29 0
 EELAYER END
 $Descr A4 11693 8268
@@
 $EndComp
 $Comp
-L power:GND #PWR0101
+L Phote_Big-rescue:GND-power #PWR0101
 U 1 1 5CADC2F2
 P 3200 1800
@@
 P 2700 2650
 F 0 "R1" V 2508 2650 40  0000 C CNN
-F 1 "120" V 2584 2650 40  0000 C CNN
+F 1 "240" V 2584 2650 40  0000 C CNN
 F 2 "Resistor_SMD:R_0603_1608Metric_Pad1.05x0.95mm_HandSolder" V 2630 2650 30  0001 C CNN
 F 3 "" H 2700 2650 30  0000 C CNN
@@
 $EndComp
 $Comp
-L power:GND #PWR0103
+L Phote_Big-rescue:GND-power #PWR0103
 U 1 1 5CADFB5E
 P 2850 3050
@@
 	3900 2650 3850 2650
 $Comp
-L power:GND #PWR0105
+L Phote_Big-rescue:GND-power #PWR0105
 U 1 1 5CAE088A
 P 3900 2950
